File: lofence.kicad_pcb (KiCad board)
At the start: 2 copper layers, 72 x 138 mm, 58 parts, among them J1 Fence+, J2 Fence-, J3 ISP, J4 DEBUG LA, J5 DEBUG LED, J6 DEBUG MCU, SW1 RESET, U1 TLV9062, U3 ATmega328PB-AU, U4 LA66, U5 MCP1253-33X50I/MS, Y1 32768 Hz

Commit message: update layout, prepared for production
Parts:
- removed the C12 at (87.3, 81.9)
- removed the D1 at (84.7, 90.4)
- removed U5: MCP1253-33X50I/MS, Package_SO:MSOP-8_3x3mm_P0.65mm
- added C4: 1nF, Capacitor_SMD:C_0805_2012Metric_Pad1.18x1.45mm_HandSolder, F.Cu at (78.4, 85.5)
- added L1: 1.5uH, Inductor_SMD:L_1008_2520Metric_Pad1.43x2.20mm_HandSolder, F.Cu at (83.1, 79.6)
- added REF**: KiCad-Logo2_5mm_SilkScreen, Symbol:KiCad-Logo2_5mm_SilkScreen, F.Cu at (71.0, 40.3)
- added REF**: OSHW-Logo2_7.3x6mm_Copper, Symbol:OSHW-Logo2_7.3x6mm_Copper, F.Cu at (40.1, 65.7)
- added REF**: Symbol_CC-ShareAlike_CopperTop_Small, Symbol:Symbol_CC-ShareAlike_CopperTop_Small, F.Cu at (46.5, 71.9)
- added REF**: Symbol_CC-Attribution_CopperTop_Small, Symbol:Symbol_CC-Attribution_CopperTop_Small, F.Cu at (40.1, 71.9)
- added U1: TPS63051RMW, ALITECS:TPS63051RMW, F.Cu at (82.8, 84.3)
- C1: renamed from C13; footprint Capacitor_SMD:C_1206_3216Metric_Pad1.33x1.80mm_HandSolder -> Capacitor_SMD:C_0805_2012Metric_Pad1.18x1.45mm_HandSolder
- C2: renamed from C14; footprint Capacitor_SMD:C_1206_3216Metric_Pad1.33x1.80mm_HandSolder -> Capacitor_SMD:C_0805_2012Metric_Pad1.18x1.45mm_HandSolder
- C3: renamed from C4; footprint Capacitor_SMD:CP_Elec_4x5.4 -> Capacitor_SMD:C_0805_2012Metric_Pad1.18x1.45mm_HandSolder
- D3, D5: value GREEN -> EMERALD
- D4, D6: value ORANGE -> YELLOW
- MH1, MH2, MH3: footprint MountingHole:MountingHole_2.7mm_M2.5 -> MountingHole:MountingHole_3.2mm_M3_DIN965_Pad
- R1, R4: value 10M 6KV -> 10M 10KV
- R10, R5, R6: footprint Resistor_SMD:R_0805_2012Metric_Pad1.20x1.40mm_HandSolder -> Resistor_SMD:R_0603_1608Metric_Pad0.98x0.95mm_HandSolder
- R11: renamed from R12; footprint Resistor_SMD:R_0805_2012Metric_Pad1.20x1.40mm_HandSolder -> Resistor_SMD:R_0603_1608Metric_Pad0.98x0.95mm_HandSolder
- R12: renamed from R16; footprint Resistor_SMD:R_0805_2012Metric_Pad1.20x1.40mm_HandSolder -> Resistor_SMD:R_0603_1608Metric_Pad0.98x0.95mm_HandSolder
- R13: renamed from R17; footprint Resistor_SMD:R_0805_2012Metric_Pad1.20x1.40mm_HandSolder -> Resistor_SMD:R_0603_1608Metric_Pad0.98x0.95mm_HandSolder
- R14: renamed from R18; footprint Resistor_SMD:R_0805_2012Metric_Pad1.20x1.40mm_HandSolder -> Resistor_SMD:R_0603_1608Metric_Pad0.98x0.95mm_HandSolder
- R15: renamed from R19; footprint Resistor_SMD:R_0805_2012Metric_Pad1.20x1.40mm_HandSolder -> Resistor_SMD:R_0603_1608Metric_Pad0.98x0.95mm_HandSolder
- R16: renamed from R20; footprint Resistor_SMD:R_0805_2012Metric_Pad1.20x1.40mm_HandSolder -> Resistor_SMD:R_0603_1608Metric_Pad0.98x0.95mm_HandSolder
- R17: renamed from R8; value 60R -> 100R; footprint Resistor_SMD:R_0805_2012Metric_Pad1.20x1.40mm_HandSolder -> Resistor_SMD:R_0603_1608Metric_Pad0.98x0.95mm_HandSolder
- R18: renamed from R11; value 60R -> 100R; footprint Resistor_SMD:R_0805_2012Metric_Pad1.20x1.40mm_HandSolder -> Resistor_SMD:R_0603_1608Metric_Pad0.98x0.95mm_HandSolder
- R19: renamed from R13; value 60R -> 100R; footprint Resistor_SMD:R_0805_2012Metric_Pad1.20x1.40mm_HandSolder -> Resistor_SMD:R_0603_1608Metric_Pad0.98x0.95mm_HandSolder
- R20: renamed from R14; value 60R -> 100R; footprint Resistor_SMD:R_0805_2012Metric_Pad1.20x1.40mm_HandSolder -> Resistor_SMD:R_0603_1608Metric_Pad0.98x0.95mm_HandSolder
- R21: renamed from R15; footprint Resistor_SMD:R_0805_2012Metric_Pad1.20x1.40mm_HandSolder -> Resistor_SMD:R_0603_1608Metric_Pad0.98x0.95mm_HandSolder
- R7: renamed from R21; footprint Resistor_SMD:R_0805_2012Metric_Pad1.20x1.40mm_HandSolder -> Resistor_SMD:R_0603_1608Metric_Pad0.98x0.95mm_HandSolder
- R8: renamed from R9; footprint Resistor_SMD:R_0805_2012Metric_Pad1.20x1.40mm_HandSolder -> Resistor_SMD:R_0603_1608Metric_Pad0.98x0.95mm_HandSolder
- R9: renamed from R7; footprint Resistor_SMD:R_0805_2012Metric_Pad1.20x1.40mm_HandSolder -> Resistor_SMD:R_0603_1608Metric_Pad0.98x0.95mm_HandSolder
- moved R7 11.6 mm to (82.6, 88.5), turned to 90 degrees
- moved U4 10.6 mm to (50.5, 48.4)
- moved J102 10.5 mm to (37.5, 151.5)
- moved J101 10.5 mm to (104.5, 151.5)
- moved C7 10.4 mm to (65.9, 54.4)
- moved C3 8.19 mm to (87.1, 84.3)
- moved C2 7.23 mm to (78.4, 78.0)
- moved R8 3.21 mm to (93.9, 67.6), turned to 180 degrees
- moved C5 2.82 mm to (92.8, 63.2)
- moved C1 2.62 mm to (78.4, 81.3), turned to 180 degrees
- moved R5 1.07 mm to (68.4, 82.3)
- moved R6 1.02 mm to (71.9, 80.3)
- moved C11 0.66 mm to (80.4, 69.1)
- moved MH2 0.50 mm to (42.0, 162.2)
- moved MH3 0.50 mm to (100.0, 162.2)
- renumbered C1 to C10, C10 to C11, C11 to C12, C6 to C5, C5 to C6, C8 to C7, C9 to C8, C7 to C9, D2 to D1, D8 to D2, J5 to J1, J1 to J101, J2 to J102, J3 to J2, J6 to J3, U1 to U2
Connections:
- BT1 pad 1: Net-(BT1-+) -> BAT_VCC
- BT2 pad 1: Net-(BT1-+) -> BAT_VCC
- C2 pad 1: BAT_VCC -> +3V3
- C3 pad 1: +3V3 -> BAT_VCC
- R7 pad 1: Net-(U5-PGOOD) -> +3V3
- R7 pad 2: +3V3 -> Net-(U1-PG)
Routing:
- net BAT_VCC: track 26.3 -> 78.1 mm
- net Net-(BT1-+): track 43.7 -> 0.00 mm
- net LA_RX: track 65.6 -> 76.5 mm
- net LA_TX: track 60.9 -> 71.8 mm
- net RN_RESET: track 29.0 -> 39.6 mm
- net Net-(J101-Pin_1): track 17.5 -> 8.25 mm
- net Net-(J102-Pin_1): track 17.2 -> 8.25 mm
- net +3V3: track 208.9 -> 202.4 mm, vias 1 -> 2
- net Net-(U1-L1): track 0.00 -> 3.79 mm
- net Net-(U1-L2): track 0.00 -> 3.79 mm
- net Net-(U5-C+): track 3.19 -> 0.00 mm
- net Net-(U5-C-): track 3.18 -> 0.00 mm
- net Net-(U5-PGOOD): track 2.93 -> 0.00 mm
- net Net-(U1-SS): track 0.00 -> 2.67 mm
- net Net-(U1-PG): track 0.00 -> 2.01 mm
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