File: LoFence-V2.kicad_pcb (KiCad board)
At the start: 2 copper layers, 72 x 138 mm, 62 parts, among them J1 DEBUG LED, J101 Fence+, J102 Fence-, J2 ISP, J3 DEBUG MCU, J4 DEBUG LA, SW1 RESET, U1 TPS63051RMW, U2 TLV9062, U3 ATmega328PB-AU, U4 LA66, Y1 32768 Hz

Commit message: rename project files and clean up
Parts:
- SW1: footprint Button_Switch_SMD:SW_SPST_B3SL-1002P -> Button_Switch_SMD:SW_SPST_Omron_B3FS-100xP
- moved SW1 0.36 mm to (99.2, 62.0)
Connections:
- net RN_RESET renamed LA_RESET
Routing:
- net +3V3: track 202.4 -> 198.2 mm
- net GND: track 75.5 -> 79.4 mm, vias 6 -> 23
- net MCU_RESET: track 46.2 -> 47.3 mm
Other:
- outline, holes or cut-outs redrawn
- board text added: "LoFence V2 REV ${REVISION} https://github.com/alex9779/lofence-v2"
- board text removed: "LoFence V2 REV A https://github.com/alex9779/lofence"

Commit message: fix TA66 rx and tx
Connections:
- U3 pad 30: LA_RX -> LA_TX
- U3 pad 31: LA_TX -> LA_RX
Changed lines of the file:
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@@
       (net 3 "MCU_RESET") (pinfunction "~{RESET}/PC6") (pintype "bidirectional"))
     (pad "30" smd rect (at -1.2 -4.25 270) (size 1.6 0.55) (layers "F.Cu" "F.Paste" "F.Mask")
-      (net 9 "LA_RX") (pinfunction "PD0") (pintype "bidirectional"))
+      (net 10 "LA_TX") (pinfunction "PD0") (pintype "bidirectional"))
     (pad "31" smd rect (at -2 -4.25 270) (size 1.6 0.55) (layers "F.Cu" "F.Paste" "F.Mask")
-      (net 10 "LA_TX") (pinfunction "PD1") (pintype "bidirectional"))
+      (net 9 "LA_RX") (pinfunction "PD1") (pintype "bidirectional"))
     (pad "32" smd rect (at -2.8 -4.25 270) (size 1.6 0.55) (layers "F.Cu" "F.Paste" "F.Mask")
       (net 41 "unconnected-(U3-PD2-Pad32)") (pinfunction "PD2") (pintype "bidirectional+no_connect"))
@@
   (segment (start 58.7064 50.0888) (end 71.374 62.7564) (width 0.25) (layer "B.Cu") (net 8))
   (segment (start 41.148 50.0888) (end 58.7064 50.0888) (width 0.25) (layer "B.Cu") (net 8))
-  (segment (start 72.2192 77.597) (end 72.2 77.5778) (width 0.25) (layer "F.Cu") (net 9))
+  (segment (start 73 77.5966) (end 72.9996 77.597) (width 0.25) (layer "F.Cu") (net 9))
   (segment (start 53.721 62.738) (end 46.2216 62.738) (width 0.25) (layer "F.Cu") (net 9))
   (segment (start 46.2216 62.738) (end 43.146 59.6624) (width 0.25) (layer "F.Cu") (net 9))
-  (segment (start 72.2 77.5778) (end 72.2 72.957) (width 0.25) (layer "F.Cu") (net 9))
   (segment (start 43.146 59.6624) (end 43.146 58.3874) (width 0.25) (layer "F.Cu") (net 9))
+  (segment (start 73 72.957) (end 73 77.5966) (width 0.25) (layer "F.Cu") (net 9))
+  (via (at 72.9996 77.597) (size 0.8) (drill 0.4) (layers "F.Cu" "B.Cu") (net 9))
   (via (at 53.721 62.738) (size 0.8) (drill 0.4) (layers "F.Cu" "B.Cu") (net 9))
-  (via (at 72.2192 77.597) (size 0.8) (drill 0.4) (layers "F.Cu" "B.Cu") (net 9))
-  (segment (start 72.2192 77.597) (end 68.58 77.597) (width 0.25) (layer "B.Cu") (net 9))
-  (segment (start 87.357 92.049) (end 98.0135 92.049) (width 0.25) (layer "B.Cu") (net 9))
-  (segment (start 68.58 77.597) (end 53.721 62.738) (width 0.25) (layer "B.Cu") (net 9))
-  (segment (start 72.2192 77.597) (end 72.905 77.597) (width 0.25) (layer "B.Cu") (net 9))
+  (segment (start 72.9996 77.597) (end 68.58 77.597) (width 0.25) (layer "B.Cu") (net 9))
   (segment (start 98.0135 92.049) (end 99.6385 90.424) (width 0.25) (layer "B.Cu") (net 9))
-  (segment (start 72.905 77.597) (end 87.357 92.049) (width 0.25) (layer "B.Cu") (net 9))
-  (segment (start 72.9812 72.9758) (end 73 72.957) (width 0.25) (layer "F.Cu") (net 10))
+  (segment (start 68.58 77.597) (end 53.721 62.738) (width 0.25) (layer "B.Cu") (net 9))
+  (segment (start 87.357 92.049) (end 98.0135 92.049) (width 0.25) (layer "B.Cu") (net 9))
+  (segment (start 72.9996 77.597) (end 87.357 92.049) (width 0.25) (layer "B.Cu") (net 9))
   (segment (start 54.864 61.595) (end 46.101 61.595) (width 0.25) (layer "F.Cu") (net 10))
-  (segment (start 72.9812 76.835) (end 72.9812 72.9758) (width 0.25) (layer "F.Cu") (net 10))
+  (segment (start 72.2122 76.835) (end 72.2 76.8228) (width 0.25) (layer "F.Cu") (net 10))
   (segment (start 44.246 59.74) (end 44.246 58.3874) (width 0.25) (layer "F.Cu") (net 10))
+  (segment (start 72.2 76.8228) (end 72.2 72.957) (width 0.25) (layer "F.Cu") (net 10))
   (segment (start 46.101 61.595) (end 44.246 59.74) (width 0.25) (layer "F.Cu") (net 10))
-  (via (at 72.9812 76.835) (size 0.8) (drill 0.4) (layers "F.Cu" "B.Cu") (net 10))
+  (via (at 72.2122 76.835) (size 0.8) (drill 0.4) (layers "F.Cu" "B.Cu") (net 10))
   (via (at 54.864 61.595) (size 0.8) (drill 0.4) (layers "F.Cu" "B.Cu") (net 10))
   (segment (start 72.9812 76.835) (end 73.6295 76.835) (width 0.25) (layer "B.Cu") (net 10))
   (segment (start 95.9235 91.599) (end 97.0985 90.424) (width 0.25) (layer "B.Cu") (net 10))
-  (segment (start 72.9812 76.835) (end 70.104 76.835) (width 0.25) (layer "B.Cu") (net 10))
+  (segment (start 72.9812 76.835) (end 72.2122 76.835) (width 0.25) (layer "B.Cu") (net 10))
   (segment (start 70.104 76.835) (end 54.864 61.595) (width 0.25) (layer "B.Cu") (net 10))
+  (segment (start 72.2122 76.835) (end 70.104 76.835) (width 0.25) (layer "B.Cu") (net 10))
   (segment (start 88.3935 91.599) (end 95.9235 91.599) (width 0.25) (layer "B.Cu") (net 10))
   (segment (start 73.6295 76.835) (end 88.3935 91.599) (width 0.25) (layer "B.Cu") (net 10))

Commit message: redesinged for 4 mounting holes
Parts:
- removed the REF** at (40.1, 65.7)
- removed the REF** at (46.5, 71.9)
- removed the REF** at (40.1, 71.9)
- added MH4: MountingHole, MountingHole:MountingHole_3.2mm_M3_DIN965_Pad, F.Cu at (100.0, 162.2)
- moved MH2 134.6 mm to (100.0, 40.8)
- moved MH3 58.0 mm to (42.0, 162.2)
- moved MH1 29.9 mm to (42.0, 40.8)
- moved D3 8.18 mm to (92.3, 45.9)
- moved D4 8.18 mm to (92.3, 48.9)
- moved D5 8.18 mm to (92.3, 51.9)
- moved D6 8.18 mm to (92.3, 54.9)
- moved D7 8.18 mm to (92.3, 57.9)
- moved R17 8.18 mm to (85.3, 45.9)
- moved R18 8.18 mm to (85.3, 48.9)
- moved R19 8.18 mm to (85.3, 51.9)
- moved R20 8.18 mm to (85.3, 54.9)
- moved R21 8.18 mm to (85.3, 57.9)
- moved J1 7.57 mm to (91.8, 61.9)
- moved U4 6.45 mm to (50.5, 54.9)
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Connections:
- U3 pad 10: unconnected-(U3-PD6-Pad10) -> LED_MSR
- U3 pad 11: unconnected-(U3-PD7-Pad11) -> LED_IDLE
- U3 pad 12: LA_RESET -> LED_CLK
- U3 pad 13: unconnected-(U3-PB1-Pad13) -> LA_RESET
- U3 pad 19: LED_MSR -> unconnected-(U3-PE2-Pad19)
- U3 pad 22: LED_TX -> unconnected-(U3-PE3-Pad22)
- U3 pad 3: LED_CLK -> unconnected-(U3-PE0-Pad3)
- U3 pad 6: LED_IDLE -> unconnected-(U3-PE1-Pad6)
- U3 pad 9: unconnected-(U3-PD5-Pad9) -> LED_TX
Routing:
- net +3V3: track 198.2 -> 171.9 mm, vias 2 -> 3
- net MCU_MISO: track 70.1 -> 52.9 mm
- net LED_TX: track 32.4 -> 15.6 mm, vias 2 -> 0
- net LED_MSR: track 31.2 -> 18.3 mm, vias 2 -> 0
- net LED_CLK: track 33.9 -> 23.8 mm, vias 2 -> 0
- net LED_IDLE: track 30.2 -> 21.1 mm
- net LA_RX: track 76.5 -> 70.4 mm
- net BAT_ADC: track 12.4 -> 7.72 mm
- net LA_TX: track 71.8 -> 68.5 mm
- net MCU_SCK: track 42.8 -> 39.7 mm, vias 2 -> 1
- net BAT_GND: track 6.84 -> 3.85 mm
- net LA_RESET: track 39.6 -> 37.0 mm
- net MCU_RESET: track 47.3 -> 45.4 mm, vias 2 -> 1
- net MCU_MOSI: track 51.9 -> 50.2 mm, vias 2 -> 1
- net AVCC: track 6.54 -> 5.00 mm
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Other:
- board size 72 x 138 mm -> 72 x 133 mm

Commit message: add OSHW logo
Parts:
- added REF**: OSHW-Logo_5.7x6mm_Copper, Symbol:OSHW-Logo_5.7x6mm_Copper, F.Cu at (71.0, 51.0)
Routing:
- net GND: vias 10 -> 11

Commit message: refine edges
Routing:
- net LA_RX: track 70.4 -> 71.9 mm
- net LA_TX: track 68.5 -> 70.0 mm
- net GND: vias 11 -> 13
Other:
- outline, holes or cut-outs redrawn
Changed lines of the file:
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@@
   (gr_line locked (start 71 96.5) (end 71 106.5)
     (stroke (width 0.1) (type default)) (layer "Dwgs.User"))
-  (gr_line locked (start 71 29.5) (end 71 39.5)
+  (gr_line locked (start 71 30) (end 71 40)
     (stroke (width 0.1) (type default)) (layer "Dwgs.User"))
-  (gr_line locked (start 35 168) (end 49 168)
-    (stroke (width 0.15) (type default)) (layer "Edge.Cuts"))
-  (gr_line locked (start 93 154) (end 93 168)
-    (stroke (width 0.15) (type default)) (layer "Edge.Cuts"))
-  (gr_line locked (start 87 35) (end 87 39.5)
-    (stroke (width 0.15) (type default)) (layer "Edge.Cuts"))
-  (gr_line locked (start 93 168) (end 107 168)
-    (stroke (width 0.15) (type default)) (layer "Edge.Cuts"))
-  (gr_line locked (start 49 154) (end 93 154)
-    (stroke (width 0.15) (type default)) (layer "Edge.Cuts"))
-  (gr_line locked (start 55 35) (end 35 35)
-    (stroke (width 0.15) (type default)) (layer "Edge.Cuts"))
-  (gr_line locked (start 87 39.5) (end 55 39.5)
-    (stroke (width 0.15) (type default)) (layer "Edge.Cuts"))
-  (gr_line locked (start 107 35) (end 87 35)
-    (stroke (width 0.15) (type default)) (layer "Edge.Cuts"))
-  (gr_line locked (start 55 35) (end 55 39.5)
-    (stroke (width 0.15) (type default)) (layer "Edge.Cuts"))
-  (gr_line locked (start 107 168) (end 107 35)
-    (stroke (width 0.15) (type default)) (layer "Edge.Cuts"))
-  (gr_line locked (start 49 154) (end 49 168)
-    (stroke (width 0.15) (type default)) (layer "Edge.Cuts"))
-  (gr_line locked (start 35 35) (end 35 168)
-    (stroke (width 0.15) (type default)) (layer "Edge.Cuts"))
+  (gr_arc (start 100 35) (mid 104.949747 37.050253) (end 107 42)
+    (stroke (width 0.15) (type default)) (layer "Edge.Cuts"))
+  (gr_line (start 56 154) (end 86 154)
+    (stroke (width 0.15) (type default)) (layer "Edge.Cuts"))
+  (gr_arc (start 100 168) (mid 95.050253 165.949747) (end 93 161)
+    (stroke (width 0.15) (type default)) (layer "Edge.Cuts"))
+  (gr_arc (start 42 168) (mid 37.050253 165.949747) (end 35 161)
+    (stroke (width 0.15) (type default)) (layer "Edge.Cuts"))
+  (gr_line (start 46.5 35) (end 42 35)
+    (stroke (width 0.15) (type default)) (layer "Edge.Cuts"))
+  (gr_line (start 90.5 40) (end 51.5 40)
+    (stroke (width 0.15) (type default)) (layer "Edge.Cuts"))
+  (gr_arc (start 49 161) (mid 46.949747 165.949747) (end 42 168)
+    (stroke (width 0.15) (type default)) (layer "Edge.Cuts"))
+  (gr_line (start 100 35) (end 95.5 35)
+    (stroke (width 0.15) (type default)) (layer "Edge.Cuts"))
+  (gr_arc (start 46.5 35) (mid 48.267767 35.732233) (end 49 37.5)
+    (stroke (width 0.15) (type default)) (layer "Edge.Cuts"))
+  (gr_line (start 107 161) (end 107 42)
+    (stroke (width 0.15) (type default)) (layer "Edge.Cuts"))
+  (gr_arc (start 51.5 40) (mid 49.732233 39.267767) (end 49 37.5)
+    (stroke (width 0.15) (type default)) (layer "Edge.Cuts"))
+  (gr_arc (start 49 161) (mid 51.050253 156.050253) (end 56 154)
+    (stroke (width 0.15) (type default)) (layer "Edge.Cuts"))
+  (gr_arc (start 107 161) (mid 104.949747 165.949747) (end 100 168)
+    (stroke (width 0.15) (type default)) (layer "Edge.Cuts"))
+  (gr_arc (start 35 42) (mid 37.050253 37.050253) (end 42 35)
+    (stroke (width 0.15) (type default)) (layer "Edge.Cuts"))
+  (gr_arc (start 93 37.5) (mid 93.732233 35.732233) (end 95.5 35)
+    (stroke (width 0.15) (type default)) (layer "Edge.Cuts"))
+  (gr_arc (start 86 154) (mid 90.949747 156.050253) (end 93 161)
+    (stroke (width 0.15) (type default)) (layer "Edge.Cuts"))
+  (gr_line (start 35 42) (end 35 161)
+    (stroke (width 0.15) (type default)) (layer "Edge.Cuts"))
+  (gr_arc (start 93 37.5) (mid 92.267767 39.267767) (end 90.5 40)
+    (stroke (width 0.15) (type default)) (layer "Edge.Cuts"))
+  (gr_line (start 106 91.25) (end 106 42)
+    (stroke (width 0.1) (type default)) (layer "Margin"))
+  (gr_arc (start 36 42) (mid 37.757359 37.757359) (end 42 36)
+    (stroke (width 0.1) (type default)) (layer "Margin"))
+  (gr_arc (start 106 91.25) (mid 105.12132 93.37132) (end 103 94.25)
+    (stroke (width 0.1) (type default)) (layer "Margin"))
+  (gr_arc (start 51.5 41) (mid 49.025126 39.974874) (end 48 37.5)
+    (stroke (width 0.1) (type default)) (layer "Margin"))
+  (gr_arc (start 100 36) (mid 104.242641 37.757359) (end 106 42)
+    (stroke (width 0.1) (type default)) (layer "Margin"))
+  (gr_line (start 95.75 36) (end 100 36)
+    (stroke (width 0.1) (type default)) (layer "Margin"))
+  (gr_line (start 36 42) (end 36 91.25)
+    (stroke (width 0.1) (type default)) (layer "Margin"))
+  (gr_line (start 42 36) (end 46.5 36)
+    (stroke (width 0.1) (type default)) (layer "Margin"))
+  (gr_line (start 90.75 41) (end 51.5 41)
+    (stroke (width 0.1) (type default)) (layer "Margin"))
+  (gr_arc (start 46.5 36) (mid 47.56066 36.43934) (end 48 37.5)
+    (stroke (width 0.1) (type default)) (layer "Margin"))
+  (gr_arc (start 39 94.25) (mid 36.87868 93.37132) (end 36 91.25)
+    (stroke (width 0.1) (type default)) (layer "Margin"))
+  (gr_line (start 39 94.25) (end 103 94.25)
+    (stroke (width 0.1) (type default)) (layer "Margin"))
+  (gr_arc (start 94.25 37.5) (mid 94.68934 36.43934) (end 95.75 36)
+    (stroke (width 0.1) (type default)) (layer "Margin"))
+  (gr_arc (start 94.25 37.5) (mid 93.224874 39.974874) (end 90.75 41)
+    (stroke (width 0.1) (type default)) (layer "Margin"))
   (gr_text "On" (at 102.4824 61.9506) (layer "F.SilkS")
     (effects (font (size 1.5 1.5) (thickness 0.3)))
@@
   (via (at 81.4801 85.5926) (size 0.8) (drill 0.4) (layers "F.Cu" "B.Cu") (free) (net 1))
   (via (at 70.6254 71.3746) (size 0.8) (drill 0.4) (layers "F.Cu" "B.Cu") (free) (net 1))
+  (via (at 72.644 84.074) (size 0.8) (drill 0.4) (layers "F.Cu" "B.Cu") (free) (net 1))
   (via (at 57.912 49.53) (size 0.8) (drill 0.4) (layers "F.Cu" "B.Cu") (free) (net 1))
   (via (at 52.959 74.6252) (size 0.8) (drill 0.4) (layers "F.Cu" "B.Cu") (free) (net 1))
@@
   (via (at 39.116 90.297) (size 0.8) (drill 0.4) (layers "F.Cu" "B.Cu") (net 1))
   (via (at 57.912 58.674) (size 0.8) (drill 0.4) (layers "F.Cu" "B.Cu") (free) (net 1))
+  (via (at 84.836 90.932) (size 0.8) (drill 0.4) (layers "F.Cu" "B.Cu") (free) (net 1))
   (segment (start 78.0796 82.6201) (end 80.3021 84.8426) (width 0.3) (layer "F.Cu") (net 2))
   (segment (start 80.3021 85.3426) (end 80.3021 84.8426) (width 0.3) (layer "F.Cu") (net 2))
@@
   (via (at 72.6186 77.3684) (size 0.8) (drill 0.4) (layers "F.Cu" "B.Cu") (net 9))
   (via (at 43.1546 67.0052) (size 0.8) (drill 0.4) (layers "F.Cu" "B.Cu") (net 9))
-  (segment (start 83.457395 88.5952) (end 97.5557 88.5952) (width 0.25) (layer "B.Cu") (net 9))
+  (segment (start 72.6186 80.3686) (end 80.8452 88.5952) (width 0.25) (layer "B.Cu") (net 9))
   (segment (start 72.6186 77.3684) (end 53.5178 77.3684) (width 0.25) (layer "B.Cu") (net 9))
-  (segment (start 72.6186 77.3684) (end 72.6186 77.756405) (width 0.25) (layer "B.Cu") (net 9))
+  (segment (start 80.8452 88.5952) (end 97.5557 88.5952) (width 0.25) (layer "B.Cu") (net 9))
+  (segment (start 53.5178 77.3684) (end 43.1546 67.0052) (width 0.25) (layer "B.Cu") (net 9))
+  (segment (start 72.6186 77.3684) (end 72.6186 80.3686) (width 0.25) (layer "B.Cu") (net 9))
   (segment (start 97.5557 88.5952) (end 99.6385 90.678) (width 0.25) (layer "B.Cu") (net 9))
-  (segment (start 72.6186 77.756405) (end 83.457395 88.5952) (width 0.25) (layer "B.Cu") (net 9))
-  (segment (start 53.5178 77.3684) (end 43.1546 67.0052) (width 0.25) (layer "B.Cu") (net 9))
   (segment (start 71.8254 78.0871) (end 71.8312 78.0929) (width 0.25) (layer "F.Cu") (net 10))
   (segment (start 44.246 69.1888) (end 44.246 64.839) (width 0.25) (layer "F.Cu") (net 10))
@@
   (via (at 44.2468 69.1896) (size 0.8) (drill 0.4) (layers "F.Cu" "B.Cu") (net 10))
   (via (at 71.8312 78.0929) (size 0.8) (drill 0.4) (layers "F.Cu" "B.Cu") (net 10))
+  (segment (start 71.8312 78.0929) (end 71.8312 80.5812) (width 0.25) (layer "B.Cu") (net 10))
+  (segment (start 71.8312 80.5812) (end 80.6072 89.3572) (width 0.25) (layer "B.Cu") (net 10))
   (segment (start 53.1501 78.0929) (end 44.2468 69.1896) (width 0.25) (layer "B.Cu") (net 10))
-  (segment (start 83.0955 89.3572) (end 95.7777 89.3572) (width 0.25) (layer "B.Cu") (net 10))
+  (segment (start 95.7777 89.3572) (end 97.0985 90.678) (width 0.25) (layer "B.Cu") (net 10))
   (segment (start 71.8312 78.0929) (end 53.1501 78.0929) (width 0.25) (layer "B.Cu") (net 10))
-  (segment (start 71.8312 78.0929) (end 83.0955 89.3572) (width 0.25) (layer "B.Cu") (net 10))
-  (segment (start 95.7777 89.3572) (end 97.0985 90.678) (width 0.25) (layer "B.Cu") (net 10))
+  (segment (start 80.6072 89.3572) (end 95.7777 89.3572) (width 0.25) (layer "B.Cu") (net 10))
   (segment (start 52.9586 88.946) (end 52.9586 88.803) (width 0.25) (layer "F.Cu") (net 11))
   (segment (start 64.38 143.256) (end 64.38 104.6854) (width 0.25) (layer "F.Cu") (net 11))
@@
     (connect_pads (clearance 0.508))
     (min_thickness 0.127) (filled_areas_thickness no)
-    (fill yes (thermal_gap 0.508) (thermal_bridge_width 0.508) (smoothing fillet) (radius 5))
+    (fill yes (thermal_gap 0.508) (thermal_bridge_width 0.508))
     (polygon
       (pts
-        (xy 36 94.2)
-        (xy 106 94.2)
-        (xy 106 36)
-        (xy 88 36)
-        (xy 88 40.75)
-        (xy 53.75 40.75)
-        (xy 53.75 36)
-        (xy 36 36)
+        (xy 35.5 94.2)
+        (xy 106.5 94.2)
+        (xy 106.5 35.5)
+        (xy 35.5 35.5)
       )
     )

Commit message: switch to dual battery holder with adjusted measures
Parts:
- removed BT2: Battery_Cell, ALITECS:18500HolderSMD
- BT1: footprint ALITECS:18500HolderSMD -> ALITECS:18500HolderSMD_x2_BeilaMoo
- moved BT1 11.0 mm to (71.0, 116.0)
Routing:
- net BAT_VCC: track 78.7 -> 77.8 mm
