File: LoFence-V2.kicad_pcb (KiCad board)
At the start: 2 copper layers, 72 x 133 mm, 71 parts, among them J1 Fence+, J2 Fence-, J3 ISP, J5 DEBUG MCU, J6 DEBUG LA, Q1 LBSS84LT1G, Q2 MMBT3904, U1 TPS63051RMW, U2 TLV9062, U3 ATmega328PB-AU, U4 LA66, Y1 32768 Hz

Commit message: fix Q1 orientation
Parts:
- moved Q1 1.96 mm to (85.8, 87.7), turned to 90 degrees
- moved C3 0.79 mm to (85.8, 83.8), turned to 90 degrees
Connections:
- Q1 pad 2: PM_EN -> BAT_VCC
- Q1 pad 3: BAT_VCC -> PM_EN
Routing:
- net Net-(Q1-G): track 16.7 -> 14.0 mm
Changed lines of the file:
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@@
   )
   (footprint "Capacitor_SMD:C_0805_2012Metric_Pad1.18x1.45mm_HandSolder" (layer "F.Cu")
-    (at 85.8051 84.582)
+    (at 85.7758 83.7946 90)
     (descr "Capacitor SMD 0805 (2012 Metric), square (rectangular) end terminal, IPC_7351 nominal with elongated pad for handsoldering. (Body size source: IPC-SM-782 page 76, https://www.pcb-3d.com/wordpress/wp-content/uploads/ipc-sm-782a_amendment_1_and_2.pdf, https://docs.google.com/spreadsheets/d/1BsfQQcO9C6DZCsRaXUlFlo91Tg2WpOkGARC1WS5S8t0/edit?usp=sharing), generated with kicad-footprint-generator")
     (tags "capacitor handsolder")
@@
     (property "ki_keywords" "cap capacitor")
     (attr smd)
-    (fp_text reference "C3" (at 0 -1.68) (layer "F.SilkS")
+    (fp_text reference "C3" (at 0 1.8034 90) (layer "F.SilkS")
         (effects (font (size 1 1) (thickness 0.15)))
     )
-    (fp_text value "10uF" (at 0 1.68) (layer "F.Fab")
+    (fp_text value "10uF" (at 0 1.68 90) (layer "F.Fab")
         (effects (font (size 1 1) (thickness 0.15)))
     )
-    (fp_text user "${REFERENCE}" (at 0 0) (layer "F.Fab")
+    (fp_text user "${REFERENCE}" (at 0 0 90) (layer "F.Fab")
         (effects (font (size 0.5 0.5) (thickness 0.08)))
     )
@@
     (fp_line (start 1 0.625) (end -1 0.625)
       (stroke (width 0.1) (type solid)) (layer "F.Fab"))
-    (pad "1" smd roundrect (at -1.0375 0) (size 1.175 1.45) (layers "F.Cu" "F.Paste" "F.Mask") (roundrect_rratio 0.2127659574)
+    (pad "1" smd roundrect (at -1.0375 0 90) (size 1.175 1.45) (layers "F.Cu" "F.Paste" "F.Mask") (roundrect_rratio 0.2127659574)
       (net 13 "BAT_VCC") (pintype "passive"))
-    (pad "2" smd roundrect (at 1.0375 0) (size 1.175 1.45) (layers "F.Cu" "F.Paste" "F.Mask") (roundrect_rratio 0.2127659574)
+    (pad "2" smd roundrect (at 1.0375 0 90) (size 1.175 1.45) (layers "F.Cu" "F.Paste" "F.Mask") (roundrect_rratio 0.2127659574)
       (net 1 "GND") (pintype "passive"))
     (model "${KICAD6_3DMODEL_DIR}/Capacitor_SMD.3dshapes/C_0805_2012Metric.wrl"
@@
   )
   (footprint "Package_TO_SOT_SMD:SOT-23" (layer "F.Cu")
-    (at 85.8012 89.6366 -90)
+    (at 85.8012 87.6808 90)
     (descr "SOT, 3 Pin (https://www.jedec.org/system/files/docs/to-236h.pdf variant AB), generated with kicad-footprint-generator ipc_gullwing_generator.py")
     (tags "SOT TO_SOT_SMD")
@@
     (property "ki_keywords" "P-Channel MOSFET")
     (attr smd)
-    (fp_text reference "Q1" (at -2.5908 0 -180) (layer "F.SilkS")
+    (fp_text reference "Q1" (at 0.0254 -2.413 90) (layer "F.SilkS")
         (effects (font (size 1 1) (thickness 0.15)))
     )
@@
     (fp_line (start 0.65 1.45) (end -0.65 1.45)
       (stroke (width 0.1) (type solid)) (layer "F.Fab"))
-    (pad "1" smd roundrect (at -0.9375 -0.95 270) (size 1.475 0.6) (layers "F.Cu" "F.Paste" "F.Mask") (roundrect_rratio 0.25)
+    (pad "1" smd roundrect (at -0.9375 -0.95 90) (size 1.475 0.6) (layers "F.Cu" "F.Paste" "F.Mask") (roundrect_rratio 0.25)
       (net 37 "Net-(Q1-G)") (pinfunction "G") (pintype "input"))
-    (pad "2" smd roundrect (at -0.9375 0.95 270) (size 1.475 0.6) (layers "F.Cu" "F.Paste" "F.Mask") (roundrect_rratio 0.25)
-      (net 54 "PM_EN") (pinfunction "S") (pintype "passive"))
-    (pad "3" smd roundrect (at 0.9375 0 270) (size 1.475 0.6) (layers "F.Cu" "F.Paste" "F.Mask") (roundrect_rratio 0.25)
-      (net 13 "BAT_VCC") (pinfunction "D") (pintype "passive"))
+    (pad "2" smd roundrect (at -0.9375 0.95 90) (size 1.475 0.6) (layers "F.Cu" "F.Paste" "F.Mask") (roundrect_rratio 0.25)
+      (net 13 "BAT_VCC") (pinfunction "S") (pintype "passive"))
+    (pad "3" smd roundrect (at 0.9375 0 90) (size 1.475 0.6) (layers "F.Cu" "F.Paste" "F.Mask") (roundrect_rratio 0.25)
+      (net 54 "PM_EN") (pinfunction "D") (pintype "passive"))
     (model "${KICAD6_3DMODEL_DIR}/Package_TO_SOT_SMD.3dshapes/SOT-23.wrl"
       (offset (xyz 0 0 0))
@@
   (segment (start 82.2371 90.5568) (end 82.2371 86.7776) (width 0.27) (layer "F.Cu") (net 13))
   (segment (start 68.8105 82.9056) (end 68.8067 82.9018) (width 0.27) (layer "F.Cu") (net 13))
-  (segment (start 82.2198 90.5741) (end 85.8012 90.5741) (width 0.27) (layer "F.Cu") (net 13))
   (segment (start 104.394 94.8582) (end 104.394 71.1432) (width 0.27) (layer "F.Cu") (net 13))
   (segment (start 82.2198 92.2255) (end 82.1925 92.2528) (width 0.27) (layer "F.Cu") (net 13))
-  (segment (start 82.6721 85.3426) (end 84.007 85.3426) (width 0.27) (layer "F.Cu") (net 13))
-  (segment (start 84.007 85.3426) (end 84.7676 84.582) (width 0.27) (layer "F.Cu") (net 13))
-  (segment (start 85.8012 85.6156) (end 84.7676 84.582) (width 0.27) (layer "F.Cu") (net 13))
+  (segment (start 86.7512 85.8075) (end 85.7758 84.8321) (width 0.27) (layer "F.Cu") (net 13))
+  (segment (start 104.394 94.8582) (end 89.321 94.8582) (width 0.27) (layer "F.Cu") (net 13))
+  (segment (start 89.321 94.8582) (end 86.741 92.2782) (width 0.27) (layer "F.Cu") (net 13))
+  (segment (start 85.2653 85.3426) (end 85.7758 84.8321) (width 0.27) (layer "F.Cu") (net 13))
+  (segment (start 86.7512 88.6183) (end 86.7512 85.8075) (width 0.27) (layer "F.Cu") (net 13))
   (segment (start 102.9188 69.668) (end 96.3188 69.668) (width 0.27) (layer "F.Cu") (net 13))
   (segment (start 82.2198 90.5741) (end 82.2198 92.2255) (width 0.27) (layer "F.Cu") (net 13))
-  (segment (start 85.8012 90.5741) (end 85.8012 85.6156) (width 0.27) (layer "F.Cu") (net 13))
-  (segment (start 85.8012 93.218) (end 85.8012 90.5741) (width 0.27) (layer "F.Cu") (net 13))
+  (segment (start 82.6721 85.3426) (end 85.2653 85.3426) (width 0.27) (layer "F.Cu") (net 13))
+  (segment (start 86.741 92.2782) (end 86.741 88.6285) (width 0.27) (layer "F.Cu") (net 13))
+  (segment (start 86.741 88.6285) (end 86.7512 88.6183) (width 0.27) (layer "F.Cu") (net 13))
   (segment (start 70.8406 82.9056) (end 68.8105 82.9056) (width 0.27) (layer "F.Cu") (net 13))
   (segment (start 82.2198 90.5741) (end 82.2371 90.5568) (width 0.27) (layer "F.Cu") (net 13))
+  (segment (start 82.1925 92.2528) (end 82.2179 92.2782) (width 0.27) (layer "F.Cu") (net 13))
   (segment (start 104.394 71.1432) (end 102.9188 69.668) (width 0.27) (layer "F.Cu") (net 13))
-  (segment (start 87.4414 94.8582) (end 85.8012 93.218) (width 0.27) (layer "F.Cu") (net 13))
-  (segment (start 104.394 94.8582) (end 87.4414 94.8582) (width 0.27) (layer "F.Cu") (net 13))
+  (segment (start 82.2179 92.2782) (end 86.741 92.2782) (width 0.27) (layer "F.Cu") (net 13))
   (via (at 82.2198 90.5741) (size 0.8) (drill 0.4) (layers "F.Cu" "B.Cu") (net 13))
   (via (at 70.8406 82.9056) (size 0.8) (drill 0.4) (layers "F.Cu" "B.Cu") (net 13))
@@
   (segment (start 74.8754 68.6) (end 77.5024 68.6) (width 0.2) (layer "F.Cu") (net 34))
   (segment (start 78.2066 92.2528) (end 75.7151 92.2528) (width 0.2) (layer "F.Cu") (net 37))
-  (segment (start 86.7512 92.2426) (end 86.741 92.2528) (width 0.2) (layer "F.Cu") (net 37))
   (segment (start 80.3675 92.2528) (end 78.2066 92.2528) (width 0.2) (layer "F.Cu") (net 37))
-  (segment (start 86.7512 88.6991) (end 86.7512 92.2426) (width 0.2) (layer "F.Cu") (net 37))
-  (via (at 86.741 92.2528) (size 0.8) (drill 0.4) (layers "F.Cu" "B.Cu") (net 37))
+  (segment (start 84.8614 88.6285) (end 84.8512 88.6183) (width 0.2) (layer "F.Cu") (net 37))
+  (segment (start 84.8614 90.5764) (end 84.8614 88.6285) (width 0.2) (layer "F.Cu") (net 37))
+  (via (at 84.8614 90.5764) (size 0.8) (drill 0.4) (layers "F.Cu" "B.Cu") (net 37))
   (via (at 78.2066 92.2528) (size 0.8) (drill 0.4) (layers "F.Cu" "B.Cu") (net 37))
-  (segment (start 86.741 92.2528) (end 78.2066 92.2528) (width 0.2) (layer "B.Cu") (net 37))
+  (segment (start 83.185 92.2528) (end 78.2066 92.2528) (width 0.2) (layer "B.Cu") (net 37))
+  (segment (start 84.8614 90.5764) (end 83.185 92.2528) (width 0.2) (layer "B.Cu") (net 37))
   (segment (start 80.6951 86.7356) (end 80.7371 86.7776) (width 0.2) (layer "F.Cu") (net 40))
   (segment (start 78.0796 86.7356) (end 80.6951 86.7356) (width 0.2) (layer "F.Cu") (net 40))
@@
   (segment (start 48.0706 83.185) (end 45.7496 83.185) (width 0.2) (layer "F.Cu") (net 51))
   (segment (start 45.7496 83.185) (end 45.3226 83.612) (width 0.2) (layer "F.Cu") (net 51))
-  (segment (start 84.8512 88.6991) (end 84.8512 88.0217) (width 0.2) (layer "F.Cu") (net 54))
-  (segment (start 84.8512 88.0217) (end 82.6721 85.8426) (width 0.2) (layer "F.Cu") (net 54))
+  (segment (start 85.8012 86.7433) (end 83.5728 86.7433) (width 0.2) (layer "F.Cu") (net 54))
+  (segment (start 83.5728 86.7433) (end 82.6721 85.8426) (width 0.2) (layer "F.Cu") (net 54))
   (segment (start 67.0306 85.3608) (end 67.0306 79.6544) (width 0.2) (layer "F.Cu") (net 55))
   (segment (start 68.6254 78.0596) (end 68.6254 75.65) (width 0.2) (layer "F.Cu") (net 55))

Commit message: switch Q2 to a N-MOSFET and simplify activation circuit
Parts:
- removed the D4 at (81.5, 63.5)
- removed the D5 at (67.0, 86.4)
- removed the R18 at (83.7, 63.3)
- removed the R19 at (85.3, 63.3)
- removed the R20 at (70.0, 89.8)
- added C13: 100nF, Capacitor_SMD:C_0805_2012Metric_Pad1.18x1.45mm_HandSolder, F.Cu at (75.1, 91.8)
- Q2: value MMBT3904 -> BSS138
- R18: renamed from R21; value 100k -> 1M
- moved R17 6.57 mm to (75.1, 89.9)
- moved Q2 4.99 mm to (70.4, 89.9)
- moved R18 4.77 mm to (65.8, 89.0)
- moved J3 2.77 mm to (102.2, 78.0)
- renumbered D6 to D4, D7 to D5, D8 to D6, D9 to D7, D10 to D8, R22 to R19, R23 to R20, R24 to R21, R25 to R22, R26 to R23
Connections:
- Q2 pad 1: Net-(D4-K) (its old number) -> ACTIVATE
- R18 pad 1: Net-(D4-K) (its old number) -> ACTIVATE
- locked pad 1: BAT_VCC -> Net-(Q1-G)
- locked pad 2: Net-(R18-Pad2) -> GND
Routing:
- net Net-(Q1-G): track 14.0 -> 72.2 mm, vias 2 -> 3
- net Net-(D4-K) (its old number): track 36.7 -> 0.00 mm, vias 2 -> 0
- net BAT_VCC: track 89.2 -> 57.2 mm, vias 2 -> 0
- net Net-(R18-Pad2): track 19.9 -> 0.00 mm
- net GND: track 79.4 -> 86.0 mm
- net ACTIVATE: track 10.4 -> 16.8 mm
- net Net-(D5-K): track 3.17 -> 0.00 mm
- net MCU_SCK: track 39.7 -> 42.4 mm
- net MCU_RESET: track 56.7 -> 58.9 mm
- net Net-(D4-A) (its old number): track 2.24 -> 0.00 mm
- net MCU_MISO: track 52.9 -> 55.1 mm

Commit message: change Q2 to 2N7002
Parts:
- Q2: value BSS138 -> 2N7002
Routing:
- net MCU_MISO: track 55.1 -> 52.9 mm
Changed lines of the file:
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@@
     (fp_line (start -33.492 5.3) (end -33.492 2.8)
       (stroke (width 0.12) (type solid)) (layer "F.SilkS"))
-    (fp_line (start -31.14 -13.49) (end -35.5 -13.49)
+    (fp_line (start -31.14 -14.1) (end -35.5 -14.1)
       (stroke (width 0.12) (type solid)) (layer "F.SilkS"))
-    (fp_line (start -30.7 -20.1) (end -30.7 -13.5)
+    (fp_line (start -30.7 -20.1) (end -30.7 -14.1)
       (stroke (width 0.12) (type solid)) (layer "F.SilkS"))
-    (fp_line (start -30.7 -6.35) (end -30.7 6.35)
+    (fp_line (start -30.7 -6) (end -30.7 6)
       (stroke (width 0.12) (type default)) (layer "F.SilkS"))
-    (fp_line (start -30.7 20.1) (end -30.7 13.5)
+    (fp_line (start -30.7 20.1) (end -30.7 14.1)
       (stroke (width 0.12) (type solid)) (layer "F.SilkS"))
     (fp_line (start 30.7 -20.1) (end -30.7 -20.1)
       (stroke (width 0.12) (type solid)) (layer "F.SilkS"))
-    (fp_line (start 30.7 -13.5) (end 30.7 -20.1)
+    (fp_line (start 30.7 -14.1) (end 30.7 -20.1)
       (stroke (width 0.12) (type solid)) (layer "F.SilkS"))
-    (fp_line (start 30.7 -6.35) (end 30.7 6.35)
+    (fp_line (start 30.7 -6) (end 30.7 6)
       (stroke (width 0.12) (type default)) (layer "F.SilkS"))
-    (fp_line (start 30.7 13.5) (end 30.7 20.1)
+    (fp_line (start 30.7 14.1) (end 30.7 20.1)
       (stroke (width 0.12) (type solid)) (layer "F.SilkS"))
     (fp_line (start 30.7 20.1) (end -30.7 20.1)
@@
     (fp_line (start 34.758 4.05) (end 32.258 4.05)
       (stroke (width 0.12) (type solid)) (layer "F.SilkS"))
-    (fp_line (start -36 -13.73) (end -31.09 -13.73)
+    (fp_line (start -36 -14.1) (end -31.1 -14.1)
       (stroke (width 0.05) (type solid)) (layer "F.CrtYd"))
-    (fp_line (start -36 -6.37) (end -36 -13.73)
+    (fp_line (start -36 -6) (end -36 -14.1)
       (stroke (width 0.05) (type solid)) (layer "F.CrtYd"))
-    (fp_line (start -36 6.36) (end -31.09 6.36)
+    (fp_line (start -36 6) (end -31.09 6)
       (stroke (width 0.05) (type solid)) (layer "F.CrtYd"))
-    (fp_line (start -36 13.72) (end -36 6.36)
+    (fp_line (start -36 14.1) (end -36 6)
       (stroke (width 0.05) (type solid)) (layer "F.CrtYd"))
-    (fp_line (start -31.09 -20.15) (end -31.09 -13.73)
+    (fp_line (start -31.09 -20.15) (end -31.1 -14.1)
       (stroke (width 0.05) (type solid)) (layer "F.CrtYd"))
     (fp_line (start -31.09 -20.15) (end 31.09 -20.15)
       (stroke (width 0.05) (type solid)) (layer "F.CrtYd"))
-    (fp_line (start -31.09 -6.37) (end -36 -6.37)
+    (fp_line (start -31.09 -6) (end -36 -6)
       (stroke (width 0.05) (type solid)) (layer "F.CrtYd"))
-    (fp_line (start -31.09 6.36) (end -31.09 -6.37)
+    (fp_line (start -31.09 6) (end -31.09 -6)
       (stroke (width 0.05) (type default)) (layer "F.CrtYd"))
-    (fp_line (start -31.09 13.72) (end -36 13.72)
+    (fp_line (start -31.09 14.1) (end -36 14.1)
       (stroke (width 0.05) (type solid)) (layer "F.CrtYd"))
-    (fp_line (start -31.09 20.15) (end -31.09 13.72)
+    (fp_line (start -31.09 20.15) (end -31.09 14.1)
       (stroke (width 0.05) (type solid)) (layer "F.CrtYd"))
     (fp_line (start -31.09 20.15) (end 31.09 20.15)
       (stroke (width 0.05) (type solid)) (layer "F.CrtYd"))
-    (fp_line (start 31.09 -20.15) (end 31.09 -13.73)
+    (fp_line (start 31.09 -20.15) (end 31.09 -14.1)
       (stroke (width 0.05) (type solid)) (layer "F.CrtYd"))
-    (fp_line (start 31.09 -6.37) (end 36 -6.37)
+    (fp_line (start 31.09 -6) (end 36 -6)
       (stroke (width 0.05) (type solid)) (layer "F.CrtYd"))
-    (fp_line (start 31.09 6.37) (end 31.09 -6.37)
+    (fp_line (start 31.09 6) (end 31.09 -6)
       (stroke (width 0.05) (type default)) (layer "F.CrtYd"))
-    (fp_line (start 31.09 13.73) (end 36 13.73)
+    (fp_line (start 31.09 14.1) (end 36 14.1)
       (stroke (width 0.05) (type solid)) (layer "F.CrtYd"))
-    (fp_line (start 31.09 20.15) (end 31.09 13.73)
+    (fp_line (start 31.09 20.15) (end 31.09 14.1)
       (stroke (width 0.05) (type solid)) (layer "F.CrtYd"))
-    (fp_line (start 36 -13.73) (end 31.09 -13.73)
+    (fp_line (start 36 -14.1) (end 31.09 -14.1)
       (stroke (width 0.05) (type solid)) (layer "F.CrtYd"))
-    (fp_line (start 36 -6.37) (end 36 -13.73)
+    (fp_line (start 36 -6) (end 36 -14.1)
       (stroke (width 0.05) (type solid)) (layer "F.CrtYd"))
-    (fp_line (start 36 6.37) (end 31.09 6.37)
+    (fp_line (start 36 6) (end 31.09 6)
       (stroke (width 0.05) (type solid)) (layer "F.CrtYd"))
-    (fp_line (start 36 13.73) (end 36 6.37)
+    (fp_line (start 36 14.1) (end 36 6)
       (stroke (width 0.05) (type solid)) (layer "F.CrtYd"))
     (fp_line (start -29.98 -14.8675) (end -29.98 20.03)
@@
     (fp_line (start 29.98 -20.03) (end 29.98 20.03)
       (stroke (width 0.1) (type solid)) (layer "F.Fab"))
-    (pad "" np_thru_hole circle (at -26.895 -18.705 180) (size 2.39 2.39) (drill 2.39) (layers "F&B.Cu" "*.Mask"))
-    (pad "1" smd rect (at -31.83 -10.05 180) (size 7.34 6.35) (layers "F.Cu" "F.Paste" "F.Mask")
+    (pad "" np_thru_hole circle (at -27.895 -19.005 180) (size 2.39 2.39) (drill 2.39) (layers "F&B.Cu" "*.Mask"))
+    (pad "1" smd rect (at -32.3 -10.05 180) (size 6.35 7.5) (layers "F.Cu" "F.Paste" "F.Mask")
       (net 55 "Net-(BT1-+)") (pinfunction "+") (pintype "passive"))
-    (pad "1" smd rect (at -31.83 10.05 180) (size 7.34 6.35) (layers "F.Cu" "F.Paste" "F.Mask")
+    (pad "1" smd rect (at -32.3 10.05 180) (size 6.35 7.5) (layers "F.Cu" "F.Paste" "F.Mask")
       (net 55 "Net-(BT1-+)") (pinfunction "+") (pintype "passive"))
-    (pad "2" smd rect (at 31.83 -10.05 180) (size 7.34 6.35) (layers "F.Cu" "F.Paste" "F.Mask")
+    (pad "2" smd rect (at 32.3 -10.05 180) (size 6.35 7.5) (layers "F.Cu" "F.Paste" "F.Mask")
       (net 1 "GND") (pinfunction "-") (pintype "passive"))
-    (pad "2" smd rect (at 31.83 10.05 180) (size 7.34 6.35) (layers "F.Cu" "F.Paste" "F.Mask")
+    (pad "2" smd rect (at 32.3 10.05 180) (size 6.35 7.5) (layers "F.Cu" "F.Paste" "F.Mask")
       (net 1 "GND") (pinfunction "-") (pintype "passive"))
     (model ":KICAD_ALITECS:3dmodels/BatteryHolder_2x18500.STEP"
@@
     (descr "SOT, 3 Pin (https://www.jedec.org/system/files/docs/to-236h.pdf variant AB), generated with kicad-footprint-generator ipc_gullwing_generator.py")
     (tags "SOT TO_SOT_SMD")
+    (property "JLCPCB Rotation Offset" "180")
     (property "Sheetfile" "LoFence-V2.kicad_sch")
     (property "Sheetname" "")
-    (property "ki_description" "50V Vds, 0.22A Id, N-Channel MOSFET, SOT-23")
-    (property "ki_keywords" "N-Channel MOSFET")
+    (property "ki_description" "0.115A Id, 60V Vds, N-Channel MOSFET, SOT-23")
+    (property "ki_keywords" "N-Channel Switching MOSFET")
     (attr smd)
     (fp_text reference "Q2" (at 0 -2.4) (layer "F.SilkS")
         (effects (font (size 1 1) (thickness 0.15)))
     )
-    (fp_text value "BSS138" (at 0 2.4) (layer "F.Fab")
+    (fp_text value "2N7002" (at 0 2.4) (layer "F.Fab")
         (effects (font (size 1 1) (thickness 0.15)))
     )
@@
     (fp_line (start 1 0.625) (end -1 0.625)
       (stroke (width 0.1) (type solid)) (layer "F.Fab"))
-    (pad "1" smd roundrect (at -1.0375 0 180) (size 1.175 1.45) (layers "F.Cu" "F.Paste" "F.Mask") (roundrect_rratio 0.212766)
+    (pad "1" smd roundrect (at -1.0375 0 180) (size 1.175 1.45) (layers "F.Cu" "F.Paste" "F.Mask") (roundrect_rratio 0.2127659574)
       (net 13 "BAT_VCC") (pintype "passive"))
-    (pad "2" smd roundrect (at 1.0375 0 180) (size 1.175 1.45) (layers "F.Cu" "F.Paste" "F.Mask") (roundrect_rratio 0.212766)
+    (pad "2" smd roundrect (at 1.0375 0 180) (size 1.175 1.45) (layers "F.Cu" "F.Paste" "F.Mask") (roundrect_rratio 0.2127659574)
       (net 37 "Net-(Q1-G)") (pintype "passive"))
     (model "${KICAD6_3DMODEL_DIR}/Capacitor_SMD.3dshapes/C_0805_2012Metric.wrl"
@@
   (segment (start 67.818 64.516) (end 67.8254 64.5234) (width 0.2) (layer "F.Cu") (net 20))
   (via (at 67.818 64.516) (size 0.8) (drill 0.4) (layers "F.Cu" "B.Cu") (net 20))
+  (segment (start 91.4955 64.516) (end 67.818 64.516) (width 0.2) (layer "B.Cu") (net 20))
   (segment (start 102.1635 77.956) (end 102.1635 78.869654) (width 0.2) (layer "B.Cu") (net 20))
+  (segment (start 102.1635 77.956) (end 102.1635 75.184) (width 0.2) (layer "B.Cu") (net 20))
   (segment (start 100.7985 80.234654) (end 100.7985 84.438) (width 0.2) (layer "B.Cu") (net 20))
-  (segment (start 102.1635 75.184) (end 91.4955 64.516) (width 0.2) (layer "B.Cu") (net 20))
   (segment (start 99.6385 85.598) (end 100.7985 84.438) (width 0.2) (layer "B.Cu") (net 20))
+  (segment (start 102.1635 75.184) (end 91.4955 64.516) (width 0.2) (layer "B.Cu") (net 20))
   (segment (start 102.1635 78.869654) (end 100.7985 80.234654) (width 0.2) (layer "B.Cu") (net 20))
-  (segment (start 102.1635 77.956) (end 102.1635 75.184) (width 0.2) (layer "B.Cu") (net 20))
-  (segment (start 91.4955 64.516) (end 67.818 64.516) (width 0.2) (layer "B.Cu") (net 20))
-  (segment (start 102.1635 75.749686) (end 102.1635 77.956) (width 0.2) (layer "B.Cu") (net 20))
   (segment (start 68.6254 65.4358) (end 68.6308 65.4304) (width 0.2) (layer "F.Cu") (net 21))
   (segment (start 68.6254 67.15) (end 68.6254 65.4358) (width 0.2) (layer "F.Cu") (net 21))

Commit message: increase resistors of emerald LEDs to 1k
Parts:
- R19, R21: value 220R -> 1k
Changed lines of the file:
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@@
         (effects (font (size 1 1) (thickness 0.15)))
     )
-    (fp_text value "220R" (at 0 1.43 180) (layer "F.Fab")
+    (fp_text value "1k" (at 0 1.43 180) (layer "F.Fab")
         (effects (font (size 1 1) (thickness 0.15)))
     )
@@
         (effects (font (size 1 1) (thickness 0.15)))
     )
-    (fp_text value "220R" (at 0 1.43 180) (layer "F.Fab")
-        (effects (font (size 1 1) (thickness 0.15)))
-    )
+    (fp_text value "1k" (at 0 1.43 180) (layer "F.Fab")
+        (effects (font (size 1 1) (thickness 0.15)))
+    )
