File: LoFence-V2.kicad_pcb (KiCad board)
At the start: 2 copper layers, 72 x 133 mm, 67 parts, among them J1 Fence+, J2 Fence-, J3 ISP, J5 DEBUG MCU, J6 DEBUG LA, Q1 LBSS84LT1G, Q2 2N7002, U1 TPS63051RMW, U2 TLV9062, U3 ATmega328PB-AU, U4 LA66, Y1 32768 Hz

Commit message: turn ISP connector
Parts:
- moved J3 7.93 mm to (94.6, 75.7), turned to 0 degrees
Routing:
- net MCU_RESET: track 58.9 -> 55.1 mm
- net MCU_MISO: track 52.9 -> 49.0 mm
- net +3V3: track 180.3 -> 177.0 mm
- net MCU_SCK: track 42.4 -> 40.6 mm
- net MCU_MOSI: track 50.2 -> 49.6 mm

Commit message: cleanup
- move whole power regulator VCC behind actviation circuit
- switch to battery clamps with options for 18650 and 18500 positions
Parts:
- removed BT1: Battery_Cell, ALITECS:18500HolderSMD_x2_BeilaMoo
- added B10: MY-18650-01, ALITECS:MY-18650-01, F.Cu at (47.0, 107.5)
- added B11: MY-18650-01, ALITECS:MY-18650-01, F.Cu at (95.0, 107.5)
- added B20: MY-18650-01, ALITECS:MY-18650-01, F.Cu at (47.0, 127.5)
- added B21: MY-18650-01, ALITECS:MY-18650-01, F.Cu at (95.0, 127.5)
- added B31: MY-18650-01, ALITECS:MY-18650-01, F.Cu at (80.0, 107.5)
- added B41: MY-18650-01, ALITECS:MY-18650-01, F.Cu at (80.0, 127.5)
- moved D1 0.41 mm to (104.8, 97.4)
Connections:
- C3 pad 1: BAT_VCC -> PM_VCC
- Q1 pad 3: PM_EN -> PM_VCC
- U1 pad 10: BAT_VCC -> PM_VCC
- U1 pad 11: PM_EN -> PM_VCC
- U1 pad 12: BAT_VCC -> PM_VCC
Routing:
- net Net-(B11-Pin_1): track 26.8 -> 97.0 mm
- net GND: track 86.0 -> 102.3 mm
- net BAT_VCC: track 57.2 -> 45.1 mm
- net PM_VCC: track 0.00 -> 7.11 mm
- net PM_EN: track 3.50 -> 0.00 mm
