File: LoFence-V2.kicad_sch (KiCad schematic)
At the start: 58 parts, among them J1 DEBUG LED, J101 Fence+, J102 Fence-, J2 ISP, J3 DEBUG MCU, J4 DEBUG LA, SW1 RESET, U1 TPS63051RMW, U2 TLV9062, U3 ATmega328PB-AU, U4 LA66, Y1 32768 Hz

Commit message: rename project files and clean up
Parts:
- SW1: footprint Button_Switch_SMD:SW_SPST_B3SL-1002P -> Button_Switch_SMD:SW_SPST_Omron_B3FS-100xP
Connections:
- net RN_RESET renamed LA_RESET
Other:
- title: (none) -> LoFence V2

Commit message: fix part numbers
Parts:
- C1, C2, C3, C4: JLCPCB Part # C13585 -> (none)
- C10, C11, C12, C5, C6, C7, C8, C9: JLCPCB Part # C49678 -> (none)
- U1: JLCPCB Part # (none) -> C139412
Changed lines of the file:
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@@
       (effects (font (size 1.27 1.27)) hide)
     )
-    (property "JLCPCB Part #" "C49678" (at 252.73 55.88 0)
+    (property "JLCPCB Part #" "" (at 252.73 55.88 0)
       (effects (font (size 1.27 1.27)) hide)
     )
@@
       (effects (font (size 1.27 1.27)) hide)
     )
-    (property "JLCPCB Part #" "C49678" (at 76.2 69.85 0)
+    (property "JLCPCB Part #" "" (at 76.2 69.85 0)
       (effects (font (size 1.27 1.27)) hide)
     )
@@
       (effects (font (size 1.27 1.27)) hide)
     )
-    (property "JLCPCB Part #" "C13585" (at 127 33.02 0)
+    (property "JLCPCB Part #" "" (at 127 33.02 0)
       (effects (font (size 1.27 1.27)) hide)
     )
@@
       (effects (font (size 1.27 1.27)) hide)
     )
-    (property "JLCPCB Part #" "C49678" (at 76.2 113.03 0)
+    (property "JLCPCB Part #" "" (at 76.2 113.03 0)
       (effects (font (size 1.27 1.27)) hide)
     )
@@
       (effects (font (size 1.27 1.27)) hide)
     )
-    (property "JLCPCB Part #" "C49678" (at 104.14 90.17 0)
+    (property "JLCPCB Part #" "" (at 104.14 90.17 0)
       (effects (font (size 1.27 1.27)) hide)
     )
@@
       (effects (font (size 1.27 1.27)) hide)
     )
-    (property "JLCPCB Part #" "C49678" (at 245.11 86.36 0)
+    (property "JLCPCB Part #" "" (at 245.11 86.36 0)
       (effects (font (size 1.27 1.27)) hide)
     )
@@
       (effects (font (size 1.27 1.27)) hide)
     )
-    (property "JLCPCB Part #" "C13585" (at 210.82 30.48 0)
+    (property "JLCPCB Part #" "" (at 210.82 30.48 0)
       (effects (font (size 1.27 1.27)) hide)
     )
@@
       (effects (font (size 1.27 1.27)) hide)
     )
-    (property "JLCPCB Part #" "C13585" (at 199.39 30.48 0)
+    (property "JLCPCB Part #" "" (at 199.39 30.48 0)
       (effects (font (size 1.27 1.27)) hide)
     )
@@
       (effects (font (size 1.27 1.27)) hide)
     )
-    (property "JLCPCB Part #" "C49678" (at 40.64 132.08 0)
+    (property "JLCPCB Part #" "" (at 40.64 132.08 0)
       (effects (font (size 1.27 1.27)) hide)
     )
@@
       (effects (font (size 1.27 1.27)) hide)
     )
-    (property "JLCPCB Part #" "C49678" (at 160.02 148.59 0)
+    (property "JLCPCB Part #" "" (at 160.02 148.59 0)
       (effects (font (size 1.27 1.27)) hide)
     )
@@
       (effects (font (size 1.27 1.27)) hide)
     )
-    (property "JLCPCB Part #" "C49678" (at 166.37 148.59 0)
+    (property "JLCPCB Part #" "" (at 166.37 148.59 0)
       (effects (font (size 1.27 1.27)) hide)
     )
@@
     )
     (property "TME Order #" "" (at 158.75 36.83 0)
+      (effects (font (size 1.27 1.27)) hide)
+    )
+    (property "JLCPCB Part #" "C139412" (at 158.75 36.83 0)
       (effects (font (size 1.27 1.27)) hide)
     )
@@
       (effects (font (size 1.27 1.27)) hide)
     )
-    (property "JLCPCB Part #" "C13585" (at 177.8 41.91 0)
-      (effects (font (size 1.27 1.27)) hide)
-    )
+    (property "JLCPCB Part #" "" (at 177.8 41.91 0)
+      (effects (font (size 1.27 1.27)) hide)
+    )

Commit message: add TME order numbers
Parts:
- R2: TME Order # (none) -> MGR0.25W-1M
- R3: TME Order # (none) -> RC0805FR-075K76L
Changed lines of the file:
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@@
       (effects (font (size 1.27 1.27)) hide)
     )
-    (property "TME Order #" "" (at 45.72 21.59 0)
+    (property "TME Order #" "MGR0.25W-1M" (at 45.72 21.59 0)
       (effects (font (size 1.27 1.27)) hide)
     )
@@
       (effects (font (size 1.27 1.27)) hide)
     )
-    (property "TME Order #" "" (at 55.88 21.59 0)
+    (property "TME Order #" "RC0805FR-075K76L" (at 55.88 21.59 0)
       (effects (font (size 1.27 1.27)) hide)
     )

Commit message: fix TA66 rx and tx
Connections:
- net LA_RX: now also U3.31 (PD1); no longer U3.30 (PD0)
- net LA_TX: now also U3.30 (PD0); no longer U3.31 (PD1)
Changed lines of the file:
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@@
     )
   )
-  (global_label "LA_TX" (shape input) (at 143.51 129.54 0) (fields_autoplaced)
+  (global_label "LA_RX" (shape input) (at 143.51 129.54 0) (fields_autoplaced)
     (effects (font (size 1.27 1.27)) (justify left))
-    (property "Intersheetrefs" "${INTERSHEET_REFS}" (at 151.1024 129.54 0)
+    (property "Intersheetrefs" "${INTERSHEET_REFS}" (at 151.4048 129.54 0)
       (effects (font (size 1.27 1.27)) (justify left) hide)
     )
@@
     )
   )
-  (global_label "LA_RX" (shape input) (at 143.51 127 0) (fields_autoplaced)
+  (global_label "LA_TX" (shape input) (at 143.51 127 0) (fields_autoplaced)
     (effects (font (size 1.27 1.27)) (justify left))
-    (property "Intersheetrefs" "${INTERSHEET_REFS}" (at 151.4048 127 0)
+    (property "Intersheetrefs" "${INTERSHEET_REFS}" (at 151.1024 127 0)
       (effects (font (size 1.27 1.27)) (justify left) hide)
     )

Commit message: redesinged for 4 mounting holes
Parts:
- added MH4: MountingHole, MountingHole:MountingHole_3.2mm_M3_DIN965_Pad, symbol Mechanical:MountingHole
Connections:
- net LA_RESET: now also U3.13 (PB1); no longer U3.12 (PB0)
- net LED_CLK: now also U3.12 (PB0); no longer U3.3 (PE0)
- net LED_IDLE: now also U3.11 (PD7); no longer U3.6 (PE1)
- net LED_MSR: now also U3.10 (PD6); no longer U3.19 (PE2)
- net LED_TX: now also U3.9 (PD5); no longer U3.22 (PE3)
Other:
- note added: "Conn Debug LA"
- note removed: "Conn Debug RN"
- moved on the sheet: MH1, MH2, MH3

Commit message: add OSHW logo
Changed lines of the file:
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@@
+    )
+  )
+  (symbol (lib_id "Graphic:Logo_Open_Hardware_Small") (at 272.415 130.175 0) (unit 1)
+    (in_bom no) (on_board no) (dnp no) (fields_autoplaced)
+    (property "Reference" "#SYM1" (at 272.415 123.19 0)
+      (effects (font (size 1.27 1.27)) hide)
+    )
+    (property "Value" "Logo_Open_Hardware_Small" (at 272.415 135.89 0)
+      (effects (font (size 1.27 1.27)) hide)
+    )
+    (property "Footprint" "" (at 272.415 130.175 0)
+      (effects (font (size 1.27 1.27)) hide)
+    )
+    (property "Datasheet" "~" (at 272.415 130.175 0)
+      (effects (font (size 1.27 1.27)) hide)
+    )
+    (property "Sim.Enable" "0" (at 272.415 130.175 0)
+      (effects (font (size 1.27 1.27)) hide)
+    )
+    (instances
+      (project "LoFence-V2"
+        (path "/8df399d3-3099-43b5-83f1-a83fbf65205c"
+          (reference "#SYM1") (unit 1)
+        )
+      )
     )
   )

Commit message: switch to dual battery holder with adjusted measures
Parts:
- removed BT2: Battery_Cell, ALITECS:18500HolderSMD, symbol Device:Battery_Cell
- BT1: footprint ALITECS:18500HolderSMD -> ALITECS:18500HolderSMD_x2_BeilaMoo
Changed lines of the file:
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@@
   (junction (at 154.94 91.44) (diameter 0) (color 0 0 0 0)
   )
-  (junction (at 109.22 26.67) (diameter 0) (color 0 0 0 0)
-  )
   (junction (at 68.58 104.14) (diameter 0) (color 0 0 0 0)
   )
@@
   (junction (at 127 26.67) (diameter 0) (color 0 0 0 0)
   )
-  (junction (at 95.25 40.64) (diameter 0) (color 0 0 0 0)
-  )
   (junction (at 177.8 46.99) (diameter 0) (color 0 0 0 0)
   )
@@
     (stroke (width 0) (type default))
   )
-  (wire (pts (xy 109.22 26.67) (xy 109.22 31.75))
-    (stroke (width 0) (type default))
-  )
   (wire (pts (xy 231.14 148.59) (xy 231.14 154.94))
     (stroke (width 0) (type default))
@@
     (stroke (width 0) (type default))
   )
-  (wire (pts (xy 95.25 40.64) (xy 95.25 55.88))
+  (wire (pts (xy 95.25 39.37) (xy 95.25 55.88))
     (stroke (width 0) (type default))
   )
@@
     (stroke (width 0) (type default))
   )
-  (wire (pts (xy 95.25 39.37) (xy 95.25 40.64))
-    (stroke (width 0) (type default))
-  )
   (wire (pts (xy 187.96 24.13) (xy 199.39 24.13))
     (stroke (width 0) (type default))
@@
     (stroke (width 0) (type default))
   )
-  (wire (pts (xy 95.25 40.64) (xy 109.22 40.64))
-    (stroke (width 0) (type default))
-  )
   (wire (pts (xy 199.39 34.29) (xy 199.39 40.64))
     (stroke (width 0) (type default))
@@
     (stroke (width 0) (type default))
   )
-  (wire (pts (xy 95.25 26.67) (xy 109.22 26.67))
-    (stroke (width 0) (type default))
-  )
   (wire (pts (xy 127 39.37) (xy 143.51 39.37))
     (stroke (width 0) (type default))
@@
     (stroke (width 0) (type default))
   )
-  (wire (pts (xy 109.22 39.37) (xy 109.22 40.64))
-    (stroke (width 0) (type default))
-  )
   (wire (pts (xy 154.94 93.98) (xy 156.21 93.98))
     (stroke (width 0) (type default))
@@
     (stroke (width 0) (type default))
   )
-  (wire (pts (xy 109.22 26.67) (xy 118.11 26.67))
+  (wire (pts (xy 95.25 26.67) (xy 118.11 26.67))
     (stroke (width 0) (type default))
   )
@@
       (effects (font (size 1.27 1.27)) (justify left))
     )
-    (property "Footprint" "ALITECS:18500HolderSMD" (at 95.25 35.306 90)
+    (property "Footprint" "ALITECS:18500HolderSMD_x2_BeilaMoo" (at 95.25 35.306 90)
       (effects (font (size 1.27 1.27)) hide)
     )
@@
         )
       )
-    )
-  )
-  (symbol (lib_id "Device:Battery_Cell") (at 109.22 36.83 0) (unit 1)
-    (in_bom no) (on_board yes) (dnp no)
-    (property "Reference" "BT2" (at 110.49 29.21 0)
-      (effects (font (size 1.27 1.27)) (justify left))
-    )
-    (property "Value" "Battery_Cell" (at 110.49 31.5214 0)
-      (effects (font (size 1.27 1.27)) (justify left))
-    )
-    (property "Footprint" "ALITECS:18500HolderSMD" (at 109.22 35.306 90)
-      (effects (font (size 1.27 1.27)) hide)
-    )
-    (property "Datasheet" "~" (at 109.22 35.306 90)
-      (effects (font (size 1.27 1.27)) hide)
-    )
-    (property "TME Order #" "" (at 109.22 36.83 0)
-      (effects (font (size 1.27 1.27)) hide)
-    )
-    (pin "1")
-    (pin "2")
-    (instances
-      (project "LoFence-V2"
-        (path "/8df399d3-3099-43b5-83f1-a83fbf65205c"
-          (reference "BT2") (unit 1)
-        )
-      )
