File: LoFence-V2.kicad_sch (KiCad schematic)
At the start: 58 parts, among them J1 DEBUG LED, J101 Fence+, J102 Fence-, J2 ISP, J3 DEBUG MCU, J4 DEBUG LA, SW1 RESET, U1 TPS63051RMW, U2 TLV9062, U3 ATmega328PB-AU, U4 LA66, Y1 32768 Hz

Commit message: some refactoring
- add activate circuit
- change some parts to JLCPCB basic parts
- adjusted resistors of LEDs
- add diode to prevent battery reverse polarization
Parts:
- removed D3, D5: EMERALD, LED_SMD:LED_0805_2012Metric_Pad1.15x1.40mm_HandSolder, symbol Device:LED
- removed D4, D6: YELLOW, LED_SMD:LED_0805_2012Metric_Pad1.15x1.40mm_HandSolder, symbol Device:LED
- removed D7: RED, LED_SMD:LED_0805_2012Metric_Pad1.15x1.40mm_HandSolder, symbol Device:LED
- removed J1: DEBUG LED, Connector_PinHeader_2.54mm:PinHeader_1x03_P2.54mm_Vertical, symbol Connector_Generic:Conn_01x03
- removed J2: ISP, Connector_PinHeader_2.54mm:PinHeader_2x03_P2.54mm_Vertical, symbol Connector_Generic:Conn_02x03_Odd_Even
- removed J3: DEBUG MCU, Connector_PinHeader_2.54mm:PinHeader_1x04_P2.54mm_Vertical, symbol Connector_Generic:Conn_01x04
- removed J4: DEBUG LA, Connector_PinHeader_2.54mm:PinHeader_1x04_P2.54mm_Vertical, symbol Connector_Generic:Conn_01x04
- added D1: D_Schottky, Diode_SMD:D_SMA_Handsoldering, symbol Device:D_Schottky
- added D4, D5: 1N5819WS, Diode_SMD:D_SOD-323, symbol Diode:1N5819WS
- added Q1: LBSS84LT1G, Package_TO_SOT_SMD:SOT-23, symbol Transistor_FET:BSS83P
- added Q2: MMBT3904, Package_TO_SOT_SMD:SOT-23, symbol Transistor_BJT:MMBT3904
- added SW2: ACTIVATE, ALITECS:TS-1187A-B-A-B, symbol Switch:SW_Push
- D2: renamed from D1; value BAV70LT -> BAV70; JLCPCB Part # C82479 -> C68978
- D3: renamed from D2; value BAV70LT -> BAV70; JLCPCB Part # C82479 -> C68978
- R17: value 100R -> 100k
- R18: value 100R -> 10k
- R19: value 100R -> 220k
- R20: value 100R -> 220R
- R21: value 68R -> 100k
- SW1: footprint Button_Switch_SMD:SW_SPST_Omron_B3FS-100xP -> ALITECS:TS-1187A-B-A-B; JLCPCB Part # C87038 -> C318884
- Y1: JLCPCB Part # C841881 -> C32346
- renumbered J101 to J1, J102 to J2
Connections:
- net +3V3: no longer R17.2
- net BAT_VCC: now also R17.2, D1.1 (K), Q1.3 (D), SW2.1; no longer BT1.1 (+), U1.11 (EN)
- net GND: now also R19.2, R21.2, Q2.2 (E)
- net LED_CLK: no longer R18.2
- net LED_IDLE: no longer R19.2
- net LED_MSR: no longer R20.2
- net LED_TX: no longer R21.2
- net ACTIVATE: now reaches U3.26 (PC3)
- net ACTIVATE: now also D5.2 (A)
- net at R17.1: now also Q1.1 (G), Q2.3 (C)
- net at R18.1: now also D4.2 (A)
- net at R19.1: now also R18.2, SW2.2
- net at R20.1: now also D5.1 (K)
- net at R21.1: now also R20.2, D4.1 (K), Q2.1 (B)
- net ADC+ renamed ADC_POS
- net ADC- renamed ADC_NEG
- new net: BT1.1 (+), D1.2 (A)
- new net PM_EN: Q1.2 (S), U1.11 (EN)
- no-connect marks 10 -> 8
Other:
- added sheet Connectors and Debug (LoFence-V2_Con-Dbg.kicad_sch)
- note added: "Activation"
- note removed: "Conn Debug LA"
- note removed: "Conn Debug MCU"
- note removed: "Conn ISP"
- note removed: "LED Debug"
- moved on the sheet: C7

Commit message: fix Q1 orientation
Connections:
- net BAT_VCC: now also Q1.2 (S); no longer Q1.3 (D)
- net PM_EN: now also Q1.3 (D); no longer Q1.2 (S)
Other:
- moved on the sheet: Q1
Changed lines of the file:
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@@
     )
   )
-  (symbol (lib_id "Transistor_FET:BSS83P") (at 53.086 152.908 90) (unit 1)
+  (symbol (lib_id "Transistor_FET:BSS83P") (at 53.086 152.908 270) (mirror x) (unit 1)
     (in_bom yes) (on_board yes) (dnp no)
-    (property "Reference" "Q1" (at 59.436 152.146 90)
+    (property "Reference" "Q1" (at 61.468 151.892 90)
       (effects (font (size 1.27 1.27)))
     )
-    (property "Value" "LBSS84LT1G" (at 59.436 154.686 90)
+    (property "Value" "LBSS84LT1G" (at 61.468 154.432 90)
       (effects (font (size 1.27 1.27)))
     )
-    (property "Footprint" "Package_TO_SOT_SMD:SOT-23" (at 54.991 147.828 0)
+    (property "Footprint" "Package_TO_SOT_SMD:SOT-23" (at 51.181 147.828 0)
       (effects (font (size 1.27 1.27) italic) (justify left) hide)
     )

Commit message: switch Q2 to a N-MOSFET and simplify activation circuit
Parts:
- removed D4, D5: 1N5819WS, Diode_SMD:D_SOD-323, symbol Diode:1N5819WS
- removed Q2: MMBT3904, Package_TO_SOT_SMD:SOT-23, symbol Transistor_BJT:MMBT3904
- removed R18: 10k, Resistor_SMD:R_0603_1608Metric_Pad0.98x0.95mm_HandSolder, symbol Device:R
- removed R19: 220k, Resistor_SMD:R_0603_1608Metric_Pad0.98x0.95mm_HandSolder, symbol Device:R
- removed R20: 220R, Resistor_SMD:R_0603_1608Metric_Pad0.98x0.95mm_HandSolder, symbol Device:R
- added C13: 100nF, Capacitor_SMD:C_0805_2012Metric_Pad1.18x1.45mm_HandSolder, symbol Device:C
- added Q2: BSS138, Package_TO_SOT_SMD:SOT-23, symbol Transistor_FET:BSS138
- R18: renamed from R21; value 100k -> 1M
Connections:
- net ACTIVATE: now also R18.1, Q2.1 (G)
- net BAT_VCC: now also C13.1; no longer SW2.1
- net GND: now also SW2.2, Q2.2 (S)
- net at Q1.1 (G), R17.1: now also SW2.1, C13.2, Q2.3 (D)
Other:
- moved on the sheet: Q1, R17, R18, SW2

Commit message: change Q2 to 2N7002
Parts:
- removed Q2: BSS138, Package_TO_SOT_SMD:SOT-23, symbol Transistor_FET:BSS138
- added Q2: 2N7002, Package_TO_SOT_SMD:SOT-23, symbol Transistor_FET:2N7002
Connections:
- net ACTIVATE: now also Q2.1 (G)
- net GND: now also Q2.2 (S)
- net at C13.2, Q1.1 (G), R17.1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: now also Q2.3 (D)
Changed lines of the file:
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@@
+    (stroke (width 0) (type default))
+  )
+  (wire (pts (xy 57.658 177.292) (xy 57.658 188.722))
     (stroke (width 0) (type default))
   )
@@
   )
   (wire (pts (xy 64.77 109.22) (xy 64.77 107.95))
-    (stroke (width 0) (type default))
-  )
-  (wire (pts (xy 57.658 177.292) (xy 57.658 188.722))
     (stroke (width 0) (type default))
   )
@@
     )
   )
-  (symbol (lib_id "power:GND") (at 199.39 40.64 0) (unit 1)
-    (in_bom yes) (on_board yes) (dnp no)
-    (property "Reference" "#PWR03" (at 199.39 46.99 0)
-      (effects (font (size 1.27 1.27)) hide)
-    )
-    (property "Value" "GND" (at 199.517 45.0342 0)
-      (effects (font (size 1.27 1.27)))
-    )
-    (property "Footprint" "" (at 199.39 40.64 0)
-      (effects (font (size 1.27 1.27)) hide)
-    )
-    (property "Datasheet" "" (at 199.39 40.64 0)
-      (effects (font (size 1.27 1.27)) hide)
-    )
-    (pin "1")
-    (instances
-      (project "LoFence-V2"
-        (path "/8df399d3-3099-43b5-83f1-a83fbf65205c"
-          (reference "#PWR03") (unit 1)
-        )
-      )
-    )
-  )
-  (symbol (lib_id "Transistor_FET:BSS138") (at 60.198 172.212 0) (mirror y) (unit 1)
-    (in_bom yes) (on_board yes) (dnp no)
-    (property "Reference" "Q2" (at 53.848 170.942 0)
-      (effects (font (size 1.27 1.27)) (justify left))
-    )
-    (property "Value" "BSS138" (at 53.848 173.482 0)
+  (symbol (lib_id "Transistor_FET:2N7002") (at 60.198 172.212 0) (mirror y) (unit 1)
+    (in_bom yes) (on_board yes) (dnp no)
+    (property "Reference" "Q2" (at 54.61 173.482 0)
+      (effects (font (size 1.27 1.27)) (justify left))
+    )
+    (property "Value" "2N7002" (at 54.61 170.942 0)
       (effects (font (size 1.27 1.27)) (justify left))
     )
@@
       (effects (font (size 1.27 1.27) italic) (justify left) hide)
     )
-    (property "Datasheet" "https://www.onsemi.com/pub/Collateral/BSS138-D.PDF" (at 60.198 172.212 0)
-      (effects (font (size 1.27 1.27)) (justify left) hide)
+    (property "Datasheet" "https://www.onsemi.com/pub/Collateral/NDS7002A-D.PDF" (at 60.198 172.212 0)
+      (effects (font (size 1.27 1.27)) (justify left) hide)
+    )
+    (property "JLCPCB Rotation Offset" "180" (at 60.198 172.212 0)
+      (effects (font (size 1.27 1.27)) hide)
     )
     (pin "1")
@@
         )
       )
+    )
+  )
+  (symbol (lib_id "power:GND") (at 199.39 40.64 0) (unit 1)
+    (in_bom yes) (on_board yes) (dnp no)
+    (property "Reference" "#PWR03" (at 199.39 46.99 0)
+      (effects (font (size 1.27 1.27)) hide)
+    )
+    (property "Value" "GND" (at 199.517 45.0342 0)
+      (effects (font (size 1.27 1.27)))
+    )
+    (property "Footprint" "" (at 199.39 40.64 0)
+      (effects (font (size 1.27 1.27)) hide)
+    )
+    (property "Datasheet" "" (at 199.39 40.64 0)
+      (effects (font (size 1.27 1.27)) hide)
+    )
+    (pin "1")
+    (instances
+      (project "LoFence-V2"
+        (path "/8df399d3-3099-43b5-83f1-a83fbf65205c"
+          (reference "#PWR03") (unit 1)
+        )
+      )

Commit message: exclude holes and fence terminals from BOM
Parts:
- J1, J2, MH1, MH2, MH3, MH4: now left out of the parts list
Changed lines of the file:
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@@
   )
   (symbol (lib_id "Connector_Generic:Conn_01x01") (at 24.13 21.59 180) (unit 1)
-    (in_bom yes) (on_board yes) (dnp no)
+    (in_bom no) (on_board yes) (dnp no)
     (property "Reference" "J1" (at 26.67 25.4 0)
       (effects (font (size 1.27 1.27)) (justify left) hide)
@@
   )
   (symbol (lib_id "Connector_Generic:Conn_01x01") (at 77.47 21.59 0) (unit 1)
-    (in_bom yes) (on_board yes) (dnp no)
+    (in_bom no) (on_board yes) (dnp no)
     (property "Reference" "J2" (at 76.2 25.4 0)
       (effects (font (size 1.27 1.27)) (justify left) hide)
@@
   )
   (symbol (lib_id "Mechanical:MountingHole") (at 265.43 154.94 0) (unit 1)
-    (in_bom yes) (on_board yes) (dnp no)
+    (in_bom no) (on_board yes) (dnp no)
     (property "Reference" "MH3" (at 267.97 153.7716 0)
       (effects (font (size 1.27 1.27)) (justify left))
@@
   )
   (symbol (lib_id "Mechanical:MountingHole") (at 265.43 144.78 0) (unit 1)
-    (in_bom yes) (on_board yes) (dnp no)
+    (in_bom no) (on_board yes) (dnp no)
     (property "Reference" "MH1" (at 267.97 143.6116 0)
       (effects (font (size 1.27 1.27)) (justify left))
@@
   )
   (symbol (lib_id "Mechanical:MountingHole") (at 265.43 149.86 0) (unit 1)
-    (in_bom yes) (on_board yes) (dnp no)
+    (in_bom no) (on_board yes) (dnp no)
     (property "Reference" "MH2" (at 267.97 148.6916 0)
       (effects (font (size 1.27 1.27)) (justify left))
@@
   )
   (symbol (lib_id "Mechanical:MountingHole") (at 265.43 160.02 0) (unit 1)
-    (in_bom yes) (on_board yes) (dnp no)
+    (in_bom no) (on_board yes) (dnp no)
     (property "Reference" "MH4" (at 267.97 158.8516 0)
       (effects (font (size 1.27 1.27)) (justify left))
