File: LoFence-V2.kicad_sch (KiCad schematic)
At the start: 51 parts, among them J1 Fence+, J2 Fence-, Q1 LBSS84LT1G, Q2 2N7002, SW1 RESET, SW2 ACTIVATE, U1 TPS63051RMW, U2 TLV9062, U3 ATmega328PB-AU, U4 LA66, Y1 32768 Hz

Commit message: cleanup
- move whole power regulator VCC behind actviation circuit
- switch to battery clamps with options for 18650 and 18500 positions
Parts:
- added B10, B11, B20, B21, B31, B41: MY-18650-01, ALITECS:MY-18650-01, symbol Connector_Generic:Conn_01x01
Connections:
- net BAT_VCC: no longer C3.1, U1.10 (ILIM0), U1.12 (VIN)
- net GND: now also B10.1 (Pin_1), B20.1 (Pin_1)
- net at BT1.1 (+), D1.2 (A): now also B11.1 (Pin_1), B21.1 (Pin_1), B31.1 (Pin_1), B41.1 (Pin_1)
- net PM_EN renamed PM_VCC
- net PM_VCC: now also C3.1, U1.10 (ILIM0), U1.12 (VIN)
Other:
- moved on the sheet: BT1
