File: LoFence-V2_Con-Dbg.kicad_sch (KiCad schematic)
At the start: 14 parts, among them J1 DEBUG LED, J2 ISP, J3 DEBUG MCU, J4 DEBUG LA

Commit message: increase resistors of emerald LEDs to 1k
Parts:
- R17, R19: value 220R -> 1k
Changed lines of the file:
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@@
       (effects (font (size 1.27 1.27)))
     )
-    (property "Value" "220R" (at 84.836 20.6756 90)
+    (property "Value" "1k" (at 84.836 20.6756 90)
       (effects (font (size 1.27 1.27)))
     )
@@
       (effects (font (size 1.27 1.27)))
     )
-    (property "Value" "220R" (at 84.836 38.4556 90)
-      (effects (font (size 1.27 1.27)))
-    )
+    (property "Value" "1k" (at 84.836 38.4556 90)
+      (effects (font (size 1.27 1.27)))
+    )
