File: LoFence.kicad_pcb (KiCad board)
At the start: 2 copper layers, 72 x 133 mm, 72 parts, among them J1 Fence+, J2 Fence-, J3 ISP, J5 DEBUG MCU, J6 DEBUG LA, Q1 LBSS84LT1G, Q2 2N7002, U1 TPS63051RMW, U2 TLV9062, U3 ATmega328PB-AU, U4 LA66, Y1 32768 Hz

Commit message: allow easier LA66 firmware update
- pushing reset also resets LA66 (pulls RST low)
- optional pin header to bridge PA2/BOOT with RX
Parts:
- added J7: FLASH LA, Connector_PinHeader_2.54mm:PinHeader_1x02_P2.54mm_Vertical, F.Cu at (40.0, 73.4)
Connections:
- C5 pad 1: MCU_RESET -> LA_RESET
- J3 pad 5: MCU_RESET -> LA_RESET
- R8 pad 2: MCU_RESET -> LA_RESET
- U3 pad 29: MCU_RESET -> LA_RESET
- locked pad 1: MCU_RESET -> LA_RESET
Routing:
- net LA_RESET: track 37.5 -> 107.2 mm, vias 2 -> 5
- net MCU_RESET: track 55.1 -> 0.00 mm, vias 1 -> 0
- net LA_BOOT: track 0.00 -> 37.1 mm, vias 0 -> 1
- net LA_RX: track 71.9 -> 79.7 mm
Other:
- board text added: "FLASH"
