File: LoFence.kicad_pcb (KiCad board)
At the start: 2 copper layers, 72 x 133 mm, 73 parts, among them J1 Fence+, J2 Fence-, J3 ISP, J5 DEBUG MCU, J6 DEBUG LA, J7 FLASH LA, Q1 LBSS84LT1G, Q2 2N7002, U1 TPS63051RMW, U2 TLV9062, U3 ATmega328PB-AU, U4 LA66, Y1 32768 Hz

Commit message: adjust diode and battery clip positions
Parts:
- moved B31 3.16 mm to (77.0, 106.5)
- moved B41 3.16 mm to (77.0, 128.5)
- moved D1 1.25 mm to (98.0, 95.2)
- moved B10 1.00 mm to (47.0, 106.5)
- moved B11 1.00 mm to (95.0, 106.5)
- moved B20 1.00 mm to (47.0, 128.5)
- moved B21 1.00 mm to (95.0, 128.5)
Routing:
- net Net-(B11-Pin_1): track 100.0 -> 108.7 mm
- net BAT_VCC: track 36.5 -> 36.0 mm
Changed lines of the file:
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@@
   )
   (footprint "ALITECS:MY-18650-01" (layer "F.Cu")
-    (at 95 127.5 180)
+    (at 95 128.5 180)
     (property "JLCPCB Position Offset" "-3.8,0")
     (property "Sheetfile" "LoFence.kicad_sch")
@@
   )
   (footprint "ALITECS:MY-18650-01" (layer "F.Cu")
-    (at 47 107.5)
+    (at 47 106.5)
     (property "JLCPCB Position Offset" "-3.8,0")
     (property "Sheetfile" "LoFence.kicad_sch")
@@
   )
   (footprint "Diode_SMD:D_SMA_Handsoldering" (layer "F.Cu")
-    (at 98 96.5)
+    (at 97.99 95.25)
     (descr "Diode SMA (DO-214AC) Handsoldering")
     (tags "Diode SMA (DO-214AC) Handsoldering")
@@
   )
   (footprint "ALITECS:MY-18650-01" (layer "F.Cu")
-    (at 80 127.5 180)
+    (at 77 128.5 180)
     (property "JLCPCB Position Offset" "-3.8,0")
     (property "Sheetfile" "LoFence.kicad_sch")
@@
   )
   (footprint "ALITECS:MY-18650-01" (layer "F.Cu")
-    (at 47 127.5)
+    (at 47 128.5)
     (property "JLCPCB Position Offset" "-3.8,0")
     (property "Sheetfile" "LoFence.kicad_sch")
@@
   )
   (footprint "ALITECS:MY-18650-01" (layer "F.Cu")
-    (at 95 107.5 180)
+    (at 95 106.5 180)
     (property "JLCPCB Position Offset" "-3.8,0")
     (property "Sheetfile" "LoFence.kicad_sch")
@@
   )
   (footprint "ALITECS:MY-18650-01" (layer "F.Cu")
-    (at 80 107.5 180)
+    (at 77 106.5 180)
     (property "JLCPCB Position Offset" "-3.8,0")
     (property "Sheetfile" "LoFence.kicad_sch")
@@
     (effects (font (size 1 1) (thickness 0.15)))
   )
-  (segment (start 39.4 107.5) (end 44.5 107.5) (width 2.4) (layer "F.Cu") (net 1))
+  (segment (start 39.4 106.5) (end 39.4 91.2) (width 2.4) (layer "F.Cu") (net 1))
+  (segment (start 44.5 106.5) (end 39.4 106.5) (width 2.4) (layer "F.Cu") (net 1))
+  (segment (start 39.4 128.5) (end 44.5 128.5) (width 2.4) (layer "F.Cu") (net 1))
   (segment (start 81.2301 85.8426) (end 81.4801 85.5926) (width 0.27) (layer "F.Cu") (net 1))
-  (segment (start 47 132.464) (end 57.792 143.256) (width 2.4) (layer "F.Cu") (net 1))
   (segment (start 81.4801 85.5926) (end 81.7371 85.3356) (width 0.27) (layer "F.Cu") (net 1))
-  (segment (start 44.5 107.5) (end 47 105) (width 2.4) (layer "F.Cu") (net 1))
   (segment locked (start 62.38 143.256) (end 57.792 143.256) (width 1.2) (layer "F.Cu") (net 1))
-  (segment (start 44.5 107.5) (end 47 110) (width 2.4) (layer "F.Cu") (net 1))
+  (segment (start 39.4 106.5) (end 39.4 128.5) (width 2.4) (layer "F.Cu") (net 1))
   (segment (start 71 71) (end 70.6254 71.3746) (width 0.27) (layer "F.Cu") (net 1))
-  (segment (start 39.4 107.5) (end 39.4 127.5) (width 2.4) (layer "F.Cu") (net 1))
-  (segment (start 47 130) (end 47 132.464) (width 2.4) (layer "F.Cu") (net 1))
+  (segment (start 44.5 106.5) (end 47 104) (width 2.4) (layer "F.Cu") (net 1))
   (segment (start 70.2 71.8) (end 70.6254 71.3746) (width 0.27) (layer "F.Cu") (net 1))
   (segment (start 74.8754 71) (end 71 71) (width 0.27) (layer "F.Cu") (net 1))
+  (segment (start 44.5 128.5) (end 47 126) (width 2.4) (layer "F.Cu") (net 1))
   (segment (start 81.4801 85.5926) (end 81.7371 85.8496) (width 0.27) (layer "F.Cu") (net 1))
+  (segment (start 57.792 141.792) (end 57.792 143.256) (width 2.4) (layer "F.Cu") (net 1))
   (segment (start 80.3021 85.8426) (end 81.2301 85.8426) (width 0.27) (layer "F.Cu") (net 1))
-  (segment (start 44.5 127.5) (end 47 130) (width 2.4) (layer "F.Cu") (net 1))
   (segment (start 81.7371 85.3356) (end 81.7371 84.4076) (width 0.27) (layer "F.Cu") (net 1))
+  (segment (start 47 131) (end 57.792 141.792) (width 2.4) (layer "F.Cu") (net 1))
   (segment (start 66.3754 71.8) (end 70.2 71.8) (width 0.27) (layer "F.Cu") (net 1))
-  (segment (start 39.4 107.5) (end 39.4 91.2) (width 2.4) (layer "F.Cu") (net 1))
-  (segment (start 44.5 127.5) (end 47 125) (width 2.4) (layer "F.Cu") (net 1))
+  (segment (start 44.5 106.5) (end 47 109) (width 2.4) (layer "F.Cu") (net 1))
+  (segment (start 47 131) (end 44.5 128.5) (width 2.4) (layer "F.Cu") (net 1))
   (segment (start 81.7371 85.8496) (end 81.7371 86.7776) (width 0.27) (layer "F.Cu") (net 1))
-  (segment (start 39.4 127.5) (end 44.5 127.5) (width 2.4) (layer "F.Cu") (net 1))
   (segment (start 102.9188 65.968) (end 96.3188 65.968) (width 0.2) (layer "F.Cu") (net 1))
   (via (at 39.4 91.2) (size 0.8) (drill 0.4) (layers "F.Cu" "B.Cu") (net 1))
@@
   (segment (start 69.4254 80.4581) (end 68.8067 81.0768) (width 0.2) (layer "F.Cu") (net 11))
   (segment (start 69.4254 75.65) (end 69.4254 80.4581) (width 0.2) (layer "F.Cu") (net 11))
+  (segment (start 95.49 95.25) (end 90.2208 95.25) (width 0.27) (layer "F.Cu") (net 12))
   (segment (start 76.1707 90.0664) (end 76.0457 89.9414) (width 0.27) (layer "F.Cu") (net 12))
-  (segment (start 91.4708 96.5) (end 86.741 91.7702) (width 0.27) (layer "F.Cu") (net 12))
-  (segment (start 95.5 96.5) (end 91.4708 96.5) (width 0.27) (layer "F.Cu") (net 12))
   (segment (start 76.1707 91.7702) (end 76.1707 90.0664) (width 0.27) (layer "F.Cu") (net 12))
   (segment (start 86.741 88.6285) (end 86.7512 88.6183) (width 0.27) (layer "F.Cu") (net 12))
@@
   (segment (start 86.741 91.7702) (end 86.741 88.6285) (width 0.27) (layer "F.Cu") (net 12))
   (segment (start 76.1707 91.7702) (end 86.741 91.7702) (width 0.27) (layer "F.Cu") (net 12))
+  (segment (start 90.2208 95.25) (end 86.741 91.7702) (width 0.27) (layer "F.Cu") (net 12))
   (segment (start 70.2254 78.6347) (end 70.8387 79.248) (width 0.2) (layer "F.Cu") (net 13))
   (segment (start 70.2254 75.65) (end 70.2254 78.6347) (width 0.2) (layer "F.Cu") (net 13))
@@
   (segment (start 69.4103 89.0016) (end 69.4205 88.9914) (width 0.2) (layer "F.Cu") (net 53))
   (segment (start 66.7493 81.88656) (end 66.7493 89.0016) (width 0.2) (layer "F.Cu") (net 53))
-  (segment (start 97.5 127.5) (end 95 125) (width 0.27) (layer "F.Cu") (net 54))
-  (segment (start 80 130) (end 82.5 127.5) (width 0.27) (layer "F.Cu") (net 54))
-  (segment (start 102.6 98.95) (end 102.6 107.5) (width 0.27) (layer "F.Cu") (net 54))
-  (segment (start 82.5 107.5) (end 80 105) (width 0.27) (layer "F.Cu") (net 54))
-  (segment (start 102.6 107.5) (end 102.6 127.5) (width 0.27) (layer "F.Cu") (net 54))
-  (segment (start 87.6 107.5) (end 97.5 107.5) (width 0.27) (layer "F.Cu") (net 54))
-  (segment (start 97.5 127.5) (end 102.6 127.5) (width 0.27) (layer "F.Cu") (net 54))
-  (segment (start 100.5 96.85) (end 102.6 98.95) (width 0.27) (layer "F.Cu") (net 54))
-  (segment (start 82.5 127.5) (end 87.6 127.5) (width 0.27) (layer "F.Cu") (net 54))
-  (segment (start 87.6 127.5) (end 97.5 127.5) (width 0.27) (layer "F.Cu") (net 54))
-  (segment (start 102.6 107.5) (end 97.5 107.5) (width 0.27) (layer "F.Cu") (net 54))
-  (segment (start 82.5 107.5) (end 80 110) (width 0.27) (layer "F.Cu") (net 54))
-  (segment (start 95 110) (end 97.5 107.5) (width 0.27) (layer "F.Cu") (net 54))
-  (segment (start 95 130) (end 97.5 127.5) (width 0.27) (layer "F.Cu") (net 54))
-  (segment (start 87.6 107.5) (end 82.5 107.5) (width 0.27) (layer "F.Cu") (net 54))
-  (segment (start 97.5 107.5) (end 95 105) (width 0.27) (layer "F.Cu") (net 54))
-  (segment (start 82.5 127.5) (end 80 125) (width 0.27) (layer "F.Cu") (net 54))
+  (segment (start 84.6 106.5) (end 79.5 106.5) (width 0.27) (layer "F.Cu") (net 54))
+  (segment (start 79.5 128.5) (end 77 126) (width 0.27) (layer "F.Cu") (net 54))
+  (segment (start 95 109) (end 97.425 106.575) (width 0.27) (layer "F.Cu") (net 54))
+  (segment (start 97.5 106.5) (end 102.6 106.5) (width 0.27) (layer "F.Cu") (net 54))
+  (segment (start 102.6 128.5) (end 97.5 128.5) (width 0.27) (layer "F.Cu") (net 54))
+  (segment (start 102.6 97.36) (end 102.6 128.5) (width 0.27) (layer "F.Cu") (net 54))
+  (segment (start 84.6 128.5) (end 79.5 128.5) (width 0.27) (layer "F.Cu") (net 54))
+  (segment (start 95 104) (end 97.425 106.425) (width 0.27) (layer "F.Cu") (net 54))
+  (segment (start 97.5 128.5) (end 95 126) (width 0.27) (layer "F.Cu") (net 54))
+  (segment (start 79.5 128.5) (end 77 131) (width 0.27) (layer "F.Cu") (net 54))
+  (segment (start 100.49 95.25) (end 102.6 97.36) (width 0.27) (layer "F.Cu") (net 54))
+  (segment (start 79.5 106.5) (end 77 104) (width 0.27) (layer "F.Cu") (net 54))
+  (segment (start 97.5 106.5) (end 84.6 106.5) (width 0.27) (layer "F.Cu") (net 54))
+  (segment (start 97.425 106.575) (end 97.425 106.425) (width 0.27) (layer "F.Cu") (net 54))
+  (segment (start 97.5 128.5) (end 84.6 128.5) (width 0.27) (layer "F.Cu") (net 54))
+  (segment (start 97.425 106.425) (end 97.5 106.5) (width 0.27) (layer "F.Cu") (net 54))
+  (segment (start 79.5 106.5) (end 77 109) (width 0.27) (layer "F.Cu") (net 54))
+  (segment (start 95 131) (end 97.5 128.5) (width 0.27) (layer "F.Cu") (net 54))
   (segment (start 52.546 47.4098) (end 52.546 44.889) (width 0.2) (layer "F.Cu") (net 56))
   (segment (start 52.5596 47.4234) (end 52.546 47.4098) (width 0.2) (layer "F.Cu") (net 56))

Commit message: change D1
Parts:
- D1: value D_Schottky -> SS54
Changed lines of the file:
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@@
     (descr "Diode SMA (DO-214AC) Handsoldering")
     (tags "Diode SMA (DO-214AC) Handsoldering")
-    (property "JLCPCB Part #" "C412437")
+    (property "JLCPCB Part #" "")
     (property "JLCPCB Position Offset" "")
     (property "Sheetfile" "LoFence.kicad_sch")
@@
         (effects (font (size 1 1) (thickness 0.15)))
     )
-    (fp_text value "D_Schottky" (at 0 2.6) (layer "F.Fab")
+    (fp_text value "SS54" (at 0 2.6) (layer "F.Fab")
         (effects (font (size 1 1) (thickness 0.15)))
     )

Commit message: change R5 and R6 to some more common and higher values to reduce measuring current
this change has been done to all rev0.4 devices manually
Parts:
- R5, R6: value 232R -> 100k
Changed lines of the file:
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@@
     (descr "Resistor SMD 0603 (1608 Metric), square (rectangular) end terminal, IPC_7351 nominal with elongated pad for handsoldering. (Body size source: IPC-SM-782 page 72, https://www.pcb-3d.com/wordpress/wp-content/uploads/ipc-sm-782a_amendment_1_and_2.pdf), generated with kicad-footprint-generator")
     (tags "resistor handsolder")
-    (property "JLCPCB Part #" "C22913")
+    (property "JLCPCB Part #" "")
     (property "JLCPCB Position Offset" "")
     (property "Sheetfile" "LoFence.kicad_sch")
@@
         (effects (font (size 1 1) (thickness 0.15)))
     )
-    (fp_text value "232R" (at 0 1.43 -90) (layer "F.Fab")
+    (fp_text value "100k" (at 0 1.43 -90) (layer "F.Fab")
         (effects (font (size 1 1) (thickness 0.15)))
     )
@@
     (descr "Resistor SMD 0603 (1608 Metric), square (rectangular) end terminal, IPC_7351 nominal with elongated pad for handsoldering. (Body size source: IPC-SM-782 page 72, https://www.pcb-3d.com/wordpress/wp-content/uploads/ipc-sm-782a_amendment_1_and_2.pdf), generated with kicad-footprint-generator")
     (tags "resistor handsolder")
-    (property "JLCPCB Part #" "C22913")
+    (property "JLCPCB Part #" "")
     (property "JLCPCB Position Offset" "")
     (property "Sheetfile" "LoFence.kicad_sch")
@@
         (effects (font (size 1 1) (thickness 0.15)))
     )
-    (fp_text value "232R" (at 0 1.43 -90) (layer "F.Fab")
-        (effects (font (size 1 1) (thickness 0.15)))
-    )
+    (fp_text value "100k" (at 0 1.43 -90) (layer "F.Fab")
+        (effects (font (size 1 1) (thickness 0.15)))
+    )

Commit message: fix GitHub URL
Other:
- board text added: "${TITLE} REV ${REVISION} https://github.com/Alex9779/LoFence"
- board text removed: "${TITLE} REV ${REVISION} https://github.com/alex9779/lofence-v2"
Changed lines of the file:
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@@
     (effects (font (size 1 1) (thickness 0.15)) (justify left bottom))
   )
-  (gr_text "${TITLE} REV ${REVISION}\nhttps://github.com/alex9779/lofence-v2\n" (at 71 149.5) (layer "F.SilkS")
+  (gr_text "${TITLE} REV ${REVISION}\nhttps://github.com/Alex9779/LoFence\n" (at 71 149.5) (layer "F.SilkS")
     (effects (font (size 1.3 1.3) (thickness 0.25)))
   )
