File: LoFence.kicad_pcb (KiCad board)
At the start: 2 copper layers, 72 x 133 mm, 73 parts, among them J1 Fence+, J2 Fence-, J3 ISP, J5 DEBUG MCU, J6 DEBUG LA, J7 FLASH LA, Q1 LBSS84LT1G, Q2 2N7002, U1 TPS63051RMW, U2 TLV9062, U3 ATmega328PB-AU, U4 LA66, Y1 32768 Hz

Commit message: extend Flash LA connector with RST and GND
Parts:
- J7: footprint Connector_PinHeader_2.54mm:PinHeader_1x02_P2.54mm_Vertical -> Connector_PinHeader_2.54mm:PinHeader_1x04_P2.54mm_Vertical
- moved R15 4.32 mm to (40.0, 83.6)
- moved J7 4.23 mm to (40.0, 69.2), turned to 0 degrees
Connections:
- J7 pad 1: LA_RX -> LA_BOOT
- J7 pad 2: LA_BOOT -> LA_RX
Routing:
- net LA_RESET: track 37.5 -> 52.4 mm
- net LA_RX: track 79.7 -> 78.0 mm
- net LA_BOOT: track 37.1 -> 35.5 mm
Other:
- board text added: "FLASH LA"
- board text removed: "FLASH"
Changed lines of the file:
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@@
   )
   (footprint "Resistor_SMD:R_0603_1608Metric_Pad0.98x0.95mm_HandSolder" (layer "F.Cu")
-    (at 40.0046 79.294)
+    (at 40 83.61)
     (descr "Resistor SMD 0603 (1608 Metric), square (rectangular) end terminal, IPC_7351 nominal with elongated pad for handsoldering. (Body size source: IPC-SM-782 page 72, https://www.pcb-3d.com/wordpress/wp-content/uploads/ipc-sm-782a_amendment_1_and_2.pdf), generated with kicad-footprint-generator")
     (tags "resistor handsolder")
@@
     (property "ki_keywords" "R res resistor")
     (attr smd)
-    (fp_text reference "R15" (at 0 -1.43) (layer "F.SilkS")
+    (fp_text reference "R15" (at -0.01 1.51) (layer "F.SilkS")
         (effects (font (size 1 1) (thickness 0.15)))
     )
@@
     (property "ki_keywords" "cap capacitor")
     (attr smd)
-    (fp_text reference "C9" (at 0 -1.778) (layer "F.SilkS")
+    (fp_text reference "C9" (at 0.0046 1.633) (layer "F.SilkS")
         (effects (font (size 1 1) (thickness 0.15)))
     )
@@
     )
   )
-  (footprint "Connector_PinHeader_2.54mm:PinHeader_1x02_P2.54mm_Vertical" (layer "F.Cu")
-    (at 40.012 73.438 180)
-    (descr "Through hole straight pin header, 1x02, 2.54mm pitch, single row")
-    (tags "Through hole pin header THT 1x02 2.54mm single row")
+  (footprint "Connector_PinHeader_2.54mm:PinHeader_1x04_P2.54mm_Vertical" (layer "F.Cu")
+    (at 40.04 69.21)
+    (descr "Through hole straight pin header, 1x04, 2.54mm pitch, single row")
+    (tags "Through hole pin header THT 1x04 2.54mm single row")
     (property "JLCPCB Position Offset" "")
     (property "Sheetfile" "LoFence_Con-Dbg.kicad_sch")
@@
     (property "dnp" "")
     (property "exclude_from_bom" "")
-    (property "ki_description" "Generic connector, single row, 01x02, script generated (kicad-library-utils/schlib/autogen/connector/)")
+    (property "ki_description" "Generic connector, single row, 01x04, script generated (kicad-library-utils/schlib/autogen/connector/)")
     (property "ki_keywords" "connector")
     (attr through_hole exclude_from_bom)
@@
         (effects (font (size 1 1) (thickness 0.15)))
     )
-    (fp_text value "FLASH LA" (at 0 4.87) (layer "F.Fab")
+    (fp_text value "FLASH LA" (at 0 9.95) (layer "F.Fab")
         (effects (font (size 1 1) (thickness 0.15)))
     )
-    (fp_text user "${REFERENCE}" (at 0 1.27 90) (layer "F.Fab")
+    (fp_text user "${REFERENCE}" (at 0 3.81 90) (layer "F.Fab")
         (effects (font (size 1 1) (thickness 0.15)))
     )
@@
     (fp_line (start -1.33 0) (end -1.33 -1.33)
       (stroke (width 0.12) (type solid)) (layer "F.SilkS"))
-    (fp_line (start -1.33 1.27) (end -1.33 3.87)
+    (fp_line (start -1.33 1.27) (end -1.33 8.95)
       (stroke (width 0.12) (type solid)) (layer "F.SilkS"))
     (fp_line (start -1.33 1.27) (end 1.33 1.27)
       (stroke (width 0.12) (type solid)) (layer "F.SilkS"))
-    (fp_line (start -1.33 3.87) (end 1.33 3.87)
+    (fp_line (start -1.33 8.95) (end 1.33 8.95)
       (stroke (width 0.12) (type solid)) (layer "F.SilkS"))
-    (fp_line (start 1.33 1.27) (end 1.33 3.87)
+    (fp_line (start 1.33 1.27) (end 1.33 8.95)
       (stroke (width 0.12) (type solid)) (layer "F.SilkS"))
-    (fp_line (start -1.8 -1.8) (end -1.8 4.35)
+    (fp_line (start -1.8 -1.8) (end -1.8 9.4)
       (stroke (width 0.05) (type solid)) (layer "F.CrtYd"))
-    (fp_line (start -1.8 4.35) (end 1.8 4.35)
+    (fp_line (start -1.8 9.4) (end 1.8 9.4)
       (stroke (width 0.05) (type solid)) (layer "F.CrtYd"))
     (fp_line (start 1.8 -1.8) (end -1.8 -1.8)
       (stroke (width 0.05) (type solid)) (layer "F.CrtYd"))
-    (fp_line (start 1.8 4.35) (end 1.8 -1.8)
+    (fp_line (start 1.8 9.4) (end 1.8 -1.8)
       (stroke (width 0.05) (type solid)) (layer "F.CrtYd"))
     (fp_line (start -1.27 -0.635) (end -0.635 -1.27)
       (stroke (width 0.1) (type solid)) (layer "F.Fab"))
-    (fp_line (start -1.27 3.81) (end -1.27 -0.635)
+    (fp_line (start -1.27 8.89) (end -1.27 -0.635)
       (stroke (width 0.1) (type solid)) (layer "F.Fab"))
     (fp_line (start -0.635 -1.27) (end 1.27 -1.27)
       (stroke (width 0.1) (type solid)) (layer "F.Fab"))
-    (fp_line (start 1.27 -1.27) (end 1.27 3.81)
+    (fp_line (start 1.27 -1.27) (end 1.27 8.89)
       (stroke (width 0.1) (type solid)) (layer "F.Fab"))
-    (fp_line (start 1.27 3.81) (end -1.27 3.81)
+    (fp_line (start 1.27 8.89) (end -1.27 8.89)
       (stroke (width 0.1) (type solid)) (layer "F.Fab"))
-    (pad "1" thru_hole rect (at 0 0 180) (size 1.7 1.7) (drill 1) (layers "*.Cu" "*.Mask")
-      (net 8 "LA_RX") (pinfunction "Pin_1") (pintype "passive"))
-    (pad "2" thru_hole oval (at 0 2.54 180) (size 1.7 1.7) (drill 1) (layers "*.Cu" "*.Mask")
-      (net 56 "LA_BOOT") (pinfunction "Pin_2") (pintype "passive"))
-    (model "${KIPRJMOD}/packages3D/PinHeader_1x02_P2.54mm_Vertical.wrl" hide
+    (pad "1" thru_hole rect (at 0 0) (size 1.7 1.7) (drill 1) (layers "*.Cu" "*.Mask")
+      (net 56 "LA_BOOT") (pinfunction "Pin_1") (pintype "passive"))
+    (pad "2" thru_hole oval (at 0 2.54) (size 1.7 1.7) (drill 1) (layers "*.Cu" "*.Mask")
+      (net 8 "LA_RX") (pinfunction "Pin_2") (pintype "passive"))
+    (pad "3" thru_hole oval (at 0 5.08) (size 1.7 1.7) (drill 1) (layers "*.Cu" "*.Mask")
+      (net 7 "LA_RESET") (pinfunction "Pin_3") (pintype "passive"))
+    (pad "4" thru_hole oval (at 0 7.62) (size 1.7 1.7) (drill 1) (layers "*.Cu" "*.Mask")
+      (net 1 "GND") (pinfunction "Pin_4") (pintype "passive"))
+    (model "${KICAD6_3DMODEL_DIR}/Connector_PinHeader_2.54mm.3dshapes/PinHeader_1x04_P2.54mm_Vertical.wrl" hide
       (offset (xyz 0 0 0))
       (scale (xyz 1 1 1))
@@
     (effects (font (size 1.5 1.5) (thickness 0.3)))
   )
-  (gr_text "FLASH" (at 37.472 72.163 90) (layer "F.SilkS")
+  (gr_text "FLASH LA" (at 37.45 73.01 90) (layer "F.SilkS")
     (effects (font (size 1.5 1.5) (thickness 0.3)))
   )
@@
   (segment (start 59.9221 81.072) (end 65.3441 75.65) (width 0.2) (layer "F.Cu") (net 4))
   (segment (start 58.5951 81.072) (end 57.7061 80.183) (width 0.2) (layer "F.Cu") (net 4))
+  (segment (start 41.0421 81.453) (end 40.9225 81.5726) (width 0.2) (layer "F.Cu") (net 5))
   (segment (start 43.3386 81.453) (end 41.0421 81.453) (width 0.2) (layer "F.Cu") (net 5))
   (segment (start 47.777 76.4515) (end 48.0818 76.4515) (width 0.2) (layer "F.Cu") (net 5))
-  (segment (start 41.0421 79.3315) (end 41.0046 79.294) (width 0.2) (layer "F.Cu") (net 5))
   (segment (start 43.3386 81.453) (end 43.3386 80.024) (width 0.2) (layer "F.Cu") (net 5))
+  (segment (start 40.9225 81.5726) (end 40.9225 83.6) (width 0.2) (layer "F.Cu") (net 5))
   (segment (start 51.1333 73.4) (end 66.3754 73.4) (width 0.2) (layer "F.Cu") (net 5))
+  (segment (start 40.9225 83.6) (end 40.9125 83.61) (width 0.2) (layer "F.Cu") (net 5))
   (segment (start 43.3386 80.024) (end 46.9111 76.4515) (width 0.2) (layer "F.Cu") (net 5))
-  (segment (start 41.0421 81.453) (end 41.0421 79.3315) (width 0.2) (layer "F.Cu") (net 5))
   (segment (start 48.0818 76.4515) (end 51.1333 73.4) (width 0.2) (layer "F.Cu") (net 5))
   (segment (start 46.9111 76.4515) (end 47.777 76.4515) (width 0.2) (layer "F.Cu") (net 5))
@@
   (via (at 40.9194 56.515) (size 0.8) (drill 0.4) (layers "F.Cu" "B.Cu") (net 7))
   (via (at 47.244 62.865) (size 0.8) (drill 0.4) (layers "F.Cu" "B.Cu") (net 7))
+  (segment (start 46.30485 62.865) (end 42.4546 66.71525) (width 0.2) (layer "B.Cu") (net 7))
   (segment (start 47.244 62.8396) (end 40.9194 56.515) (width 0.2) (layer "B.Cu") (net 7))
+  (segment (start 42.4546 66.71525) (end 42.4546 71.8754) (width 0.2) (layer "B.Cu") (net 7))
+  (segment (start 47.244 62.865) (end 46.30485 62.865) (width 0.2) (layer "B.Cu") (net 7))
   (segment (start 47.244 62.865) (end 47.244 62.8396) (width 0.2) (layer "B.Cu") (net 7))
+  (segment (start 42.4546 71.8754) (end 40.04 74.29) (width 0.2) (layer "B.Cu") (net 7))
   (segment (start 43.1546 64.8476) (end 43.146 64.839) (width 0.2) (layer "F.Cu") (net 8))
   (segment (start 72.6186 77.3684) (end 72.6254 77.3616) (width 0.2) (layer "F.Cu") (net 8))
+  (segment (start 43.1546 67.0052) (end 43.1546 68.6354) (width 0.2) (layer "F.Cu") (net 8))
   (segment (start 43.1546 67.0052) (end 43.1546 64.8476) (width 0.2) (layer "F.Cu") (net 8))
+  (segment (start 43.1546 68.6354) (end 40.04 71.75) (width 0.2) (layer "F.Cu") (net 8))
   (segment (start 72.6254 77.3616) (end 72.6254 75.65) (width 0.2) (layer "F.Cu") (net 8))
   (via (at 72.6186 77.3684) (size 0.8) (drill 0.4) (layers "F.Cu" "B.Cu") (net 8))
@@
   (segment (start 72.6186 80.3686) (end 80.8452 88.5952) (width 0.2) (layer "B.Cu") (net 8))
   (segment (start 72.6186 77.3684) (end 53.5178 77.3684) (width 0.2) (layer "B.Cu") (net 8))
-  (segment (start 43.1546 67.0052) (end 43.1546 70.2954) (width 0.2) (layer "B.Cu") (net 8))
-  (segment (start 43.1546 70.2954) (end 40.012 73.438) (width 0.2) (layer "B.Cu") (net 8))
   (segment (start 80.8452 88.5952) (end 97.5557 88.5952) (width 0.2) (layer "B.Cu") (net 8))
   (segment (start 53.5178 77.3684) (end 43.1546 67.0052) (width 0.2) (layer "B.Cu") (net 8))
@@
   (via (at 52.5596 47.4234) (size 0.8) (drill 0.4) (layers "F.Cu" "B.Cu") (net 56))
   (segment (start 42.4504 47.4234) (end 52.5596 47.4234) (width 0.2) (layer "B.Cu") (net 56))
-  (segment (start 40.012 49.8618) (end 42.4504 47.4234) (width 0.2) (layer "B.Cu") (net 56))
-  (segment (start 40.012 70.898) (end 40.012 49.8618) (width 0.2) (layer "B.Cu") (net 56))
+  (segment (start 40.01 69.18) (end 40.01 49.8638) (width 0.2) (layer "B.Cu") (net 56))
+  (segment (start 40.01 49.8638) (end 42.4504 47.4234) (width 0.2) (layer "B.Cu") (net 56))
+  (segment (start 40.04 69.21) (end 40.01 69.18) (width 0.2) (layer "B.Cu") (net 56))
   (segment (start 82.9313 69.668) (end 82.931 69.6683) (width 0.2) (layer "F.Cu") (net 57))
   (segment (start 92.5556 69.668) (end 85.9556 69.668) (width 0.2) (layer "F.Cu") (net 57))

Commit message: switch default R3 to 5k6 --> 11.8kV and do not exclude
Parts:
- R3: value 5k76 -> 5k6
Changed lines of the file:
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@@
     (descr "Resistor SMD 0805 (2012 Metric), square (rectangular) end terminal, IPC_7351 nominal with elongated pad for handsoldering. (Body size source: IPC-SM-782 page 72, https://www.pcb-3d.com/wordpress/wp-content/uploads/ipc-sm-782a_amendment_1_and_2.pdf), generated with kicad-footprint-generator")
     (tags "resistor handsolder")
-    (property "JLCPCB Part #" "C3016502")
+    (property "JLCPCB Part #" "")
     (property "JLCPCB Position Offset" "")
     (property "Sheetfile" "LoFence.kicad_sch")
     (property "Sheetname" "")
-    (property "TME Order #" "RC0805FR-075K76L")
-    (property "exclude_from_bom" "")
+    (property "TME Order #" "")
     (property "ki_description" "Resistor")
     (property "ki_keywords" "R res resistor")
-    (attr smd exclude_from_bom)
+    (attr smd)
     (fp_text reference "R3" (at 0 -1.65) (layer "F.SilkS")
         (effects (font (size 1 1) (thickness 0.15)))
     )
-    (fp_text value "5k76" (at 0 1.65) (layer "F.Fab")
+    (fp_text value "5k6" (at 0 1.65) (layer "F.Fab")
         (effects (font (size 1 1) (thickness 0.15)))
     )
