File: LoFence_Con-Dbg.kicad_sch (KiCad schematic)
At the start: 14 parts, among them J1 DEBUG LED, J2 ISP, J3 DEBUG MCU, J4 DEBUG LA

Commit message: allow easier LA66 firmware update
- pushing reset also resets LA66 (pulls RST low)
- optional pin header to bridge PA2/BOOT with RX
Parts:
- added J?: FLASH LA, Connector_PinHeader_2.54mm:PinHeader_1x02_P2.54mm_Vertical, symbol Connector_Generic:Conn_01x02
- renumbered D3 to D?, D5 to D?, D6 to D?, D7 to D?, D4 to D?, J4 to J?, J2 to J?, J3 to J?, J1 to J?, R18 to R?, R20 to R?, R17 to R?, R21 to R?, R19 to R?
Connections:
- net LA_RX: now also J?.1 (Pin_1)
- new net LA_BOOT: J?.2 (Pin_2)
Other:
- note added: "Conn Flash LA"
- moved on the sheet: J?
