File: LoFence_Con-Dbg.kicad_sch (KiCad schematic)
At the start: 15 parts

Commit message: include LED pins in BOM
Parts:
- J?: JLCPCB Position Offset (none) -> -2.54,0; JLCPCB Rotation Offset (none) -> 90; now in the parts list
Changed lines of the file:
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@@
   )
   (symbol (lib_id "Connector_Generic:Conn_01x03") (at 108.966 32.512 90) (unit 1)
-    (in_bom no) (on_board yes) (dnp no)
+    (in_bom yes) (on_board yes) (dnp no)
     (property "Reference" "J?" (at 107.8992 30.48 0)
       (effects (font (size 1.27 1.27)) (justify left))
@@
       (effects (font (size 1.27 1.27)) hide)
     )
-    (property "JLCPCB Position Offset" "" (at 108.966 32.512 0)
+    (property "JLCPCB Position Offset" "-2.54,0" (at 108.966 32.512 0)
       (effects (font (size 1.27 1.27)) hide)
     )
+    (property "JLCPCB Rotation Offset" "90" (at 108.966 32.512 0)
+      (effects (font (size 1.27 1.27)) hide)
+    )

Commit message: extend Flash LA connector with RST and GND
Parts:
- J?: footprint Connector_PinHeader_2.54mm:PinHeader_1x02_P2.54mm_Vertical -> Connector_PinHeader_2.54mm:PinHeader_1x04_P2.54mm_Vertical; symbol Connector_Generic:Conn_01x02 -> Connector_Generic:Conn_01x04
Connections:
- net GND: now also J?.4 (Pin_4)
- net LA_BOOT: now also J?.1 (Pin_1); no longer J?.2 (Pin_2)
- net LA_RX: now also J?.2 (Pin_2); no longer J?.1 (Pin_1)
- new net LA_RESET: J?.3 (Pin_3)
Changed lines of the file:
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@@
+    (stroke (width 0) (type default))
+  )
+  (wire (pts (xy 26.924 107.95) (xy 29.464 107.95))
     (stroke (width 0) (type default))
   )
@@
     (stroke (width 0) (type default))
   )
+  (wire (pts (xy 26.924 100.33) (xy 29.464 100.33))
+    (stroke (width 0) (type default))
+  )
+  (polyline (pts (xy 42.672 40.386) (xy 15.24 40.386))
+    (stroke (width 0) (type default))
+  )
+  (polyline (pts (xy 15.24 88.646) (xy 15.24 65.786))
+    (stroke (width 0) (type default))
+  )
+  (wire (pts (xy 78.486 50.292) (xy 81.026 50.292))
+    (stroke (width 0) (type default))
+  )
+  (polyline (pts (xy 67.056 14.732) (xy 67.056 62.992))
+    (stroke (width 0) (type default))
+  )
+  (wire (pts (xy 29.464 49.276) (xy 26.924 49.276))
+    (stroke (width 0) (type default))
+  )
+  (polyline (pts (xy 15.24 114.3) (xy 15.24 91.44))
+    (stroke (width 0) (type default))
+  )
+  (wire (pts (xy 29.464 82.296) (xy 26.924 82.296))
+    (stroke (width 0) (type default))
+  )
+  (wire (pts (xy 78.486 23.622) (xy 81.026 23.622))
+    (stroke (width 0) (type default))
+  )
+  (wire (pts (xy 91.186 23.622) (xy 88.646 23.622))
+    (stroke (width 0) (type default))
+  )
+  (wire (pts (xy 101.346 50.292) (xy 98.806 50.292))
+    (stroke (width 0) (type default))
+  )
+  (wire (pts (xy 29.464 54.356) (xy 26.924 54.356))
+    (stroke (width 0) (type default))
+  )
+  (wire (pts (xy 101.346 59.182) (xy 98.806 59.182))
+    (stroke (width 0) (type default))
+  )
+  (polyline (pts (xy 115.316 14.732) (xy 115.316 62.992))
+    (stroke (width 0) (type default))
+  )
+  (wire (pts (xy 26.924 79.756) (xy 29.464 79.756))
+    (stroke (width 0) (type default))
+  )
+  (wire (pts (xy 46.99 28.702) (xy 44.45 28.702))
+    (stroke (width 0) (type default))
+  )
+  (wire (pts (xy 46.99 31.242) (xy 46.99 28.702))
+    (stroke (width 0) (type default))
+  )
+  (polyline (pts (xy 115.316 62.992) (xy 67.056 62.992))
+    (stroke (width 0) (type default))
+  )
+  (wire (pts (xy 101.346 50.292) (xy 101.346 41.402))
+    (stroke (width 0) (type default))
+  )
   (wire (pts (xy 26.924 102.87) (xy 29.464 102.87))
     (stroke (width 0) (type default))
   )
-  (polyline (pts (xy 42.672 40.386) (xy 15.24 40.386))
-    (stroke (width 0) (type default))
-  )
-  (polyline (pts (xy 15.24 88.646) (xy 15.24 65.786))
-    (stroke (width 0) (type default))
-  )
-  (wire (pts (xy 78.486 50.292) (xy 81.026 50.292))
-    (stroke (width 0) (type default))
-  )
-  (polyline (pts (xy 67.056 14.732) (xy 67.056 62.992))
-    (stroke (width 0) (type default))
-  )
-  (wire (pts (xy 29.464 49.276) (xy 26.924 49.276))
-    (stroke (width 0) (type default))
-  )
-  (polyline (pts (xy 15.24 114.3) (xy 15.24 91.44))
-    (stroke (width 0) (type default))
-  )
-  (wire (pts (xy 29.464 82.296) (xy 26.924 82.296))
-    (stroke (width 0) (type default))
-  )
-  (wire (pts (xy 78.486 23.622) (xy 81.026 23.622))
-    (stroke (width 0) (type default))
-  )
-  (wire (pts (xy 91.186 23.622) (xy 88.646 23.622))
-    (stroke (width 0) (type default))
-  )
-  (wire (pts (xy 101.346 50.292) (xy 98.806 50.292))
-    (stroke (width 0) (type default))
-  )
-  (wire (pts (xy 29.464 54.356) (xy 26.924 54.356))
-    (stroke (width 0) (type default))
-  )
-  (wire (pts (xy 101.346 59.182) (xy 98.806 59.182))
-    (stroke (width 0) (type default))
-  )
-  (polyline (pts (xy 115.316 14.732) (xy 115.316 62.992))
-    (stroke (width 0) (type default))
-  )
-  (wire (pts (xy 26.924 79.756) (xy 29.464 79.756))
-    (stroke (width 0) (type default))
-  )
-  (wire (pts (xy 46.99 28.702) (xy 44.45 28.702))
-    (stroke (width 0) (type default))
-  )
-  (wire (pts (xy 46.99 31.242) (xy 46.99 28.702))
-    (stroke (width 0) (type default))
-  )
-  (polyline (pts (xy 115.316 62.992) (xy 67.056 62.992))
-    (stroke (width 0) (type default))
-  )
-  (wire (pts (xy 101.346 50.292) (xy 101.346 41.402))
+  (wire (pts (xy 91.186 50.292) (xy 88.646 50.292))
+    (stroke (width 0) (type default))
+  )
+  (polyline (pts (xy 42.672 65.786) (xy 15.24 65.786))
+    (stroke (width 0) (type default))
+  )
+  (polyline (pts (xy 15.24 88.646) (xy 42.672 88.646))
+    (stroke (width 0) (type default))
+  )
+  (polyline (pts (xy 63.5 14.732) (xy 63.5 37.592))
+    (stroke (width 0) (type default))
+  )
+  (wire (pts (xy 108.966 55.372) (xy 108.966 37.592))
+    (stroke (width 0) (type default))
+  )
+  (wire (pts (xy 101.346 41.402) (xy 101.346 32.512))
+    (stroke (width 0) (type default))
+  )
+  (wire (pts (xy 101.346 32.512) (xy 98.806 32.512))
+    (stroke (width 0) (type default))
+  )
+  (wire (pts (xy 101.346 23.622) (xy 101.346 32.512))
+    (stroke (width 0) (type default))
+  )
+  (wire (pts (xy 26.924 77.216) (xy 29.464 77.216))
     (stroke (width 0) (type default))
   )
   (wire (pts (xy 26.924 105.41) (xy 29.464 105.41))
-    (stroke (width 0) (type default))
-  )
-  (wire (pts (xy 91.186 50.292) (xy 88.646 50.292))
-    (stroke (width 0) (type default))
-  )
-  (polyline (pts (xy 42.672 65.786) (xy 15.24 65.786))
-    (stroke (width 0) (type default))
-  )
-  (polyline (pts (xy 15.24 88.646) (xy 42.672 88.646))
-    (stroke (width 0) (type default))
-  )
-  (polyline (pts (xy 63.5 14.732) (xy 63.5 37.592))
-    (stroke (width 0) (type default))
-  )
-  (wire (pts (xy 108.966 55.372) (xy 108.966 37.592))
-    (stroke (width 0) (type default))
-  )
-  (wire (pts (xy 101.346 41.402) (xy 101.346 32.512))
-    (stroke (width 0) (type default))
-  )
-  (wire (pts (xy 101.346 32.512) (xy 98.806 32.512))
-    (stroke (width 0) (type default))
-  )
-  (wire (pts (xy 101.346 23.622) (xy 101.346 32.512))
-    (stroke (width 0) (type default))
-  )
-  (wire (pts (xy 26.924 77.216) (xy 29.464 77.216))
     (stroke (width 0) (type default))
   )
@@
     )
   )
-  (global_label "LA_BOOT" (shape input) (at 26.924 105.41 180) (fields_autoplaced)
-    (effects (font (size 1.27 1.27)) (justify right))
-    (property "Intersheetrefs" "${INTERSHEET_REFS}" (at 16.6101 105.41 0)
+  (global_label "LA_RX" (shape input) (at 26.924 102.87 180) (fields_autoplaced)
+    (effects (font (size 1.27 1.27)) (justify right))
+    (property "Intersheetrefs" "${INTERSHEET_REFS}" (at 19.0292 102.87 0)
       (effects (font (size 1.27 1.27)) (justify right) hide)
     )
@@
     )
   )
+  (global_label "LA_RESET" (shape input) (at 26.924 105.41 180) (fields_autoplaced)
+    (effects (font (size 1.27 1.27)) (justify right))
+    (property "Intersheetrefs" "${INTERSHEET_REFS}" (at 15.7636 105.41 0)
+      (effects (font (size 1.27 1.27)) (justify right) hide)
+    )
+  )
   (global_label "MCU_RX" (shape input) (at 26.924 51.816 180) (fields_autoplaced)
     (effects (font (size 1.27 1.27)) (justify right))
@@
     )
   )
-  (global_label "LA_RX" (shape input) (at 26.924 102.87 180) (fields_autoplaced)
-    (effects (font (size 1.27 1.27)) (justify right))
-    (property "Intersheetrefs" "${INTERSHEET_REFS}" (at 19.0292 102.87 0)
+  (global_label "LA_BOOT" (shape input) (at 26.924 100.33 180) (fields_autoplaced)
+    (effects (font (size 1.27 1.27)) (justify right))
+    (property "Intersheetrefs" "${INTERSHEET_REFS}" (at 16.6101 100.33 0)
       (effects (font (size 1.27 1.27)) (justify right) hide)
     )
@@
     )
   )
+  (symbol (lib_id "power:GND") (at 26.924 107.95 0) (unit 1)
+    (in_bom yes) (on_board yes) (dnp no)
+    (property "Reference" "#PWR?" (at 26.924 114.3 0)
+      (effects (font (size 1.27 1.27)) hide)
+    )
+    (property "Value" "GND" (at 27.051 112.3442 0)
+      (effects (font (size 1.27 1.27)))
+    )
+    (property "Footprint" "" (at 26.924 107.95 0)
+      (effects (font (size 1.27 1.27)) hide)
+    )
+    (property "Datasheet" "" (at 26.924 107.95 0)
+      (effects (font (size 1.27 1.27)) hide)
+    )
+    (pin "1")
+    (instances
+      (project "LoFence"
+        (path "/8df399d3-3099-43b5-83f1-a83fbf65205c"
+          (reference "#PWR?") (unit 1)
+        )
+        (path "/8df399d3-3099-43b5-83f1-a83fbf65205c/efd635f6-2055-4669-9417-4264f7a45d39"
+          (reference "#PWR043") (unit 1)
+        )
+      )
+    )
+  )
   (symbol (lib_id "Device:LED") (at 94.996 50.292 180) (unit 1)
     (in_bom yes) (on_board yes) (dnp no)
@@
     )
   )
-  (symbol (lib_id "Connector_Generic:Conn_01x02") (at 34.544 102.87 0) (unit 1)
+  (symbol (lib_id "Connector_Generic:Conn_01x04") (at 34.544 102.87 0) (unit 1)
     (in_bom no) (on_board yes) (dnp yes)
     (property "Reference" "J?" (at 37.084 105.41 90)
@@
       (effects (font (size 1.27 1.27)) (justify left))
     )
-    (property "Footprint" "Connector_PinHeader_2.54mm:PinHeader_1x02_P2.54mm_Vertical" (at 34.544 102.87 0)
+    (property "Footprint" "Connector_PinHeader_2.54mm:PinHeader_1x04_P2.54mm_Vertical" (at 34.544 102.87 0)
       (effects (font (size 1.27 1.27)) hide)
     )
@@
     (pin "1")
     (pin "2")
-    (instances
-      (project "LoFence"
+    (pin "3")
+    (pin "4")
+    (instances
+      (project "LoFence"
