File: LoFence.kicad_sch (KiCad schematic)
At the start: 57 parts, among them J1 Fence+, J2 Fence-, Q1 LBSS84LT1G, Q2 2N7002, SW1 RESET, SW2 ACTIVATE, U1 TPS63051RMW, U2 TLV9062, U3 ATmega328PB-AU, U4 LA66, Y1 32768 Hz

Commit message: allow easier LA66 firmware update
- pushing reset also resets LA66 (pulls RST low)
- optional pin header to bridge PA2/BOOT with RX
Connections:
- net MCU_RESET is gone; now on net LA_RESET: C5.1, R8.2, SW1.1, U3.29 (~{RESET}/PC6)
- new net LA_BOOT: U4.8 (PA2)
Other:
- sheet Connectors and Debug: file LoFence-V2_Con-Dbg.kicad_sch -> LoFence_Con-Dbg.kicad_sch
- moved on the sheet: C7

Commit message: change D1
Parts:
- D1: value D_Schottky -> SS54; JLCPCB Part # C412437 -> (none)
Changed lines of the file:
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@@
       (effects (font (size 1.27 1.27)))
     )
-    (property "Value" "D_Schottky" (at 102.87 23.495 0)
+    (property "Value" "SS54" (at 102.87 23.495 0)
       (effects (font (size 1.27 1.27)))
     )
@@
       (effects (font (size 1.27 1.27)) hide)
     )
-    (property "JLCPCB Part #" "C412437" (at 102.87 26.67 0)
+    (property "JLCPCB Part #" "" (at 102.87 26.67 0)
       (effects (font (size 1.27 1.27)) hide)
     )

Commit message: change R5 and R6 to some more common and higher values to reduce measuring current
this change has been done to all rev0.4 devices manually
Parts:
- R5, R6: value 232R -> 100k; JLCPCB Part # C22913 -> (none)
Changed lines of the file:
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@@
       (effects (font (size 1.27 1.27)) (justify right))
     )
-    (property "Value" "232R" (at 252.603 19.812 0)
+    (property "Value" "100k" (at 252.603 19.812 0)
       (effects (font (size 1.27 1.27)) (justify right))
     )
@@
       (effects (font (size 1.27 1.27)) hide)
     )
-    (property "JLCPCB Part #" "C22913" (at 251.46 21.59 0)
+    (property "JLCPCB Part #" "" (at 251.46 21.59 0)
       (effects (font (size 1.27 1.27)) hide)
     )
@@
       (effects (font (size 1.27 1.27)) (justify right))
     )
-    (property "Value" "232R" (at 265.303 19.812 0)
+    (property "Value" "100k" (at 265.303 19.812 0)
       (effects (font (size 1.27 1.27)) (justify right))
     )
@@
       (effects (font (size 1.27 1.27)) hide)
     )
-    (property "JLCPCB Part #" "C22913" (at 264.16 21.59 0)
+    (property "JLCPCB Part #" "" (at 264.16 21.59 0)
       (effects (font (size 1.27 1.27)) hide)
     )

Commit message: add JLCPCB part number for R3
but still excluded from BOM
Parts:
- R3: JLCPCB Part # (none) -> C3016502
Changed lines of the file:
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@@
+      (effects (font (size 1.27 1.27)) hide)
+    )
+    (property "JLCPCB Part #" "C3016502" (at 55.88 21.59 0)
       (effects (font (size 1.27 1.27)) hide)
     )

Commit message: remove LA_RESET from button because of reset loop with MCU
Connections:
- net LA_RESET: no longer C5.1, R8.2, SW1.1, U3.29 (~{RESET}/PC6)
- new net MCU_RESET: C5.1, R8.2, SW1.1, U3.29 (~{RESET}/PC6)
Changed lines of the file:
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@@
   (junction (at 199.39 24.13) (diameter 0) (color 0 0 0 0)
   )
-  (junction (at 252.73 48.006) (diameter 0) (color 0 0 0 0)
-  )
   (junction (at 210.82 24.13) (diameter 0) (color 0 0 0 0)
   )
@@
   )
   (junction (at 135.128 26.67) (diameter 0) (color 0 0 0 0)
-  )
-  (junction (at 252.73 51.054) (diameter 0) (color 0 0 0 0)
   )
   (junction (at 127 39.37) (diameter 0) (color 0 0 0 0)
@@
     (stroke (width 0) (type default))
   )
-  (wire (pts (xy 248.92 48.006) (xy 252.73 48.006))
-    (stroke (width 0) (type default))
-  )
   (wire (pts (xy 30.48 132.08) (xy 36.83 132.08))
     (stroke (width 0) (type default))
@@
     (stroke (width 0) (type default))
   )
-  (wire (pts (xy 252.73 51.054) (xy 252.73 49.53))
+  (wire (pts (xy 252.73 49.53) (xy 252.73 52.07))
     (stroke (width 0) (type default))
   )
@@
     (stroke (width 0) (type default))
   )
-  (wire (pts (xy 252.73 48.006) (xy 252.73 49.53))
-    (stroke (width 0) (type default))
-  )
   (wire (pts (xy 236.982 96.52) (xy 239.522 96.52))
     (stroke (width 0) (type default))
@@
     (stroke (width 0) (type default))
   )
-  (wire (pts (xy 252.73 51.054) (xy 252.73 52.07))
-    (stroke (width 0) (type default))
-  )
   (wire (pts (xy 68.58 50.8) (xy 68.58 63.5))
     (stroke (width 0) (type default))
@@
     (stroke (width 0) (type default))
   )
-  (wire (pts (xy 252.73 46.99) (xy 252.73 48.006))
+  (wire (pts (xy 252.73 46.99) (xy 252.73 49.53))
     (stroke (width 0) (type default))
   )
@@
     (stroke (width 0) (type default))
   )
-  (wire (pts (xy 248.92 51.054) (xy 252.73 51.054))
+  (wire (pts (xy 248.92 49.53) (xy 252.73 49.53))
     (stroke (width 0) (type default))
   )
@@
     )
   )
-  (global_label "LA_RESET" (shape input) (at 248.92 48.006 180) (fields_autoplaced)
-    (effects (font (size 1.27 1.27)) (justify right))
-    (property "Intersheetrefs" "${INTERSHEET_REFS}" (at 237.7596 48.006 0)
-      (effects (font (size 1.27 1.27)) (justify right) hide)
-    )
-  )
   (global_label "AVCC" (shape input) (at 128.27 73.66 0) (fields_autoplaced)
     (effects (font (size 1.27 1.27)) (justify left))
@@
     )
   )
-  (global_label "MCU_RESET" (shape input) (at 248.92 51.054 180) (fields_autoplaced)
+  (global_label "MCU_RESET" (shape input) (at 248.92 49.53 180) (fields_autoplaced)
     (effects (font (size 1.27 1.27)) (justify right))
-    (property "Intersheetrefs" "${INTERSHEET_REFS}" (at 235.8244 51.054 0)
+    (property "Intersheetrefs" "${INTERSHEET_REFS}" (at 235.8244 49.53 0)
       (effects (font (size 1.27 1.27)) (justify right) hide)
     )
