File: LoFence.kicad_sch (KiCad schematic)
At the start: 57 parts, among them J1 Fence+, J2 Fence-, Q1 LBSS84LT1G, Q2 2N7002, SW1 RESET, SW2 ACTIVATE, U1 TPS63051RMW, U2 TLV9062, U3 ATmega328PB-AU, U4 LA66, Y1 32768 Hz

Commit message: switch default R3 to 5k6 --> 11.8kV and do not exclude
Parts:
- R3: value 5k76 -> 5k6; JLCPCB Part # C3016502 -> (none); TME Order # RC0805FR-075K76L -> (none); now in the parts list
Changed lines of the file:
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@@
   )
   (symbol (lib_id "Device:R") (at 55.88 21.59 270) (unit 1)
-    (in_bom no) (on_board yes) (dnp no)
+    (in_bom yes) (on_board yes) (dnp no)
     (property "Reference" "R3" (at 55.88 16.3322 90)
       (effects (font (size 1.27 1.27)))
     )
-    (property "Value" "5k76" (at 55.88 18.6436 90)
+    (property "Value" "5k6" (at 55.88 18.6436 90)
       (effects (font (size 1.27 1.27)))
     )
@@
       (effects (font (size 1.27 1.27)) hide)
     )
-    (property "TME Order #" "RC0805FR-075K76L" (at 55.88 21.59 0)
+    (property "TME Order #" "" (at 55.88 21.59 0)
       (effects (font (size 1.27 1.27)) hide)
     )
@@
       (effects (font (size 1.27 1.27)) hide)
     )
-    (property "JLCPCB Part #" "C3016502" (at 55.88 21.59 0)
+    (property "JLCPCB Part #" "" (at 55.88 21.59 0)
       (effects (font (size 1.27 1.27)) hide)
     )
