File: KiCad/LoFence.kicad_sch (KiCad schematic)
At the start: 57 parts, among them J1 Fence+, J2 Fence-, Q1 LBSS84LT1G, Q2 2N7002, SW1 RESET, SW2 ACTIVATE, U1 TPS63051RMW, U2 TLV9062, U3 ATmega328PB-AU, U4 LA66, Y1 32768 Hz

Commit message: include R1, R2, R4 in BOM
Parts:
- R1, R2, R4: now in the parts list
Changed lines of the file:
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@@
   )
   (symbol (lib_id "Device:R") (at 35.56 21.59 270) (unit 1)
-    (in_bom no) (on_board yes) (dnp no)
+    (in_bom yes) (on_board yes) (dnp no)
     (property "Reference" "R1" (at 35.56 16.3322 90)
       (effects (font (size 1.27 1.27)))
@@
   )
   (symbol (lib_id "Device:R") (at 45.72 21.59 270) (unit 1)
-    (in_bom no) (on_board yes) (dnp no)
+    (in_bom yes) (on_board yes) (dnp no)
     (property "Reference" "R2" (at 45.72 16.3322 90)
       (effects (font (size 1.27 1.27)))
@@
   )
   (symbol (lib_id "Device:R") (at 66.04 21.59 270) (unit 1)
-    (in_bom no) (on_board yes) (dnp no)
+    (in_bom yes) (on_board yes) (dnp no)
     (property "Reference" "R4" (at 66.04 16.3322 90)
       (effects (font (size 1.27 1.27)))

Commit message: add order nurmber for R1/R4 and R2
Parts:
- R1, R4: JLCPCB Part # (none) -> C1364802; JLCPCB Position Offset (none) -> 10,0
- R2: JLCPCB Part # (none) -> C18816311
Changed lines of the file:
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@@
       (effects (font (size 1.27 1.27)) hide)
     )
-    (property "JLCPCB Position Offset" "" (at 35.56 21.59 0)
+    (property "JLCPCB Position Offset" "10,0" (at 35.56 21.59 0)
+      (effects (font (size 1.27 1.27)) hide)
+    )
+    (property "JLCPCB Part #" "C1364802" (at 35.56 21.59 0)
       (effects (font (size 1.27 1.27)) hide)
     )
@@
     )
     (property "JLCPCB Position Offset" "" (at 45.72 21.59 0)
+      (effects (font (size 1.27 1.27)) hide)
+    )
+    (property "JLCPCB Part #" "C18816311" (at 45.72 21.59 0)
       (effects (font (size 1.27 1.27)) hide)
     )
@@
       (effects (font (size 1.27 1.27)) hide)
     )
-    (property "JLCPCB Position Offset" "" (at 66.04 21.59 0)
+    (property "JLCPCB Position Offset" "10,0" (at 66.04 21.59 0)
       (effects (font (size 1.27 1.27)) hide)
     )
+    (property "JLCPCB Part #" "C1364802" (at 66.04 21.59 0)
+      (effects (font (size 1.27 1.27)) hide)
+    )
