File: KiCad/LoFence_Con-Dbg.kicad_sch (KiCad schematic)
At the start: 15 parts

Commit message: connector updates
- move connectors a little to the inside
- populate ISP connector
Parts:
- J?: JLCPCB Position Offset (none) -> -2.54,-1.27; JLCPCB Rotation Offset (none) -> 90; now fitted; now in the parts list
Changed lines of the file:
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@@
   )
   (symbol (lib_id "Connector_Generic:Conn_02x03_Odd_Even") (at 36.83 26.162 0) (unit 1)
-    (in_bom no) (on_board yes) (dnp yes)
+    (in_bom yes) (on_board yes) (dnp no)
     (property "Reference" "J?" (at 38.1 18.1102 0)
       (effects (font (size 1.27 1.27)))
@@
       (effects (font (size 1.27 1.27)) hide)
     )
-    (property "JLCPCB Position Offset" "" (at 36.83 26.162 0)
+    (property "JLCPCB Position Offset" "-2.54,-1.27" (at 36.83 26.162 0)
       (effects (font (size 1.27 1.27)) hide)
     )
+    (property "JLCPCB Rotation Offset" "90" (at 36.83 26.162 0)
+      (effects (font (size 1.27 1.27)) hide)
+    )
