File: KiCad/LoFence.kicad_pcb (KiCad board)
At the start: 2 copper layers, 72 x 133 mm, 73 parts, among them J1 Fence+, J2 Fence-, J3 ISP, J5 DEBUG MCU, J6 DEBUG LA, J7 FLASH LA, Q1 LBSS84LT1G, Q2 2N7002, U1 TPS63051RMW, U2 TLV9062, U3 ATmega328PB-AU, U4 LA66, Y1 32768 Hz

Commit message: move logo and title text to copper layer, fix DRC
Parts:
- REF**: value KiCad-Logo2_5mm_SilkScreen -> KiCad-Logo2_5mm_Copper; footprint Symbol:KiCad-Logo2_5mm_SilkScreen -> Symbol:KiCad-Logo2_5mm_Copper
- moved REF** 0.40 mm to (71.0, 44.1)
- moved REF** 0.40 mm to (71.0, 50.6)
Changed lines of the file:
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@@
     )
   )
-  (footprint "Symbol:KiCad-Logo2_5mm_SilkScreen" locked (layer "F.Cu")
-    (at 71 44.5)
+  (footprint "Symbol:KiCad-Logo2_5mm_Copper" locked (layer "F.Cu")
+    (at 71 44.1)
     (descr "KiCad Logo")
     (tags "Logo KiCad")
@@
         (effects (font (size 1 1) (thickness 0.15)))
     )
-    (fp_text value "KiCad-Logo2_5mm_SilkScreen" (at 0 5.08) (layer "F.Fab") hide
+    (fp_text value "KiCad-Logo2_5mm_Copper" (at 0 5.08) (layer "F.Fab") hide
         (effects (font (size 1 1) (thickness 0.15)))
     )
@@
         (xy 4.188614 2.275877)
       )
-      (stroke (width 0.01) (type solid)) (fill solid) (layer "F.SilkS"))
+      (stroke (width 0.01) (type solid)) (fill solid) (layer "F.Cu"))
     (fp_poly
       (pts
@@
         (xy -2.923822 2.291645)
       )
-      (stroke (width 0.01) (type solid)) (fill solid) (layer "F.SilkS"))
+      (stroke (width 0.01) (type solid)) (fill solid) (layer "F.Cu"))
     (fp_poly
       (pts
@@
         (xy -2.273043 -2.973429)
       )
-      (stroke (width 0.01) (type solid)) (fill solid) (layer "F.SilkS"))
+      (stroke (width 0.01) (type solid)) (fill solid) (layer "F.Cu"))
     (fp_poly
       (pts
@@
         (xy 4.963065 2.269163)
       )
-      (stroke (width 0.01) (type solid)) (fill solid) (layer "F.SilkS"))
+      (stroke (width 0.01) (type solid)) (fill solid) (layer "F.Cu"))
     (fp_poly
       (pts
@@
         (xy 6.228823 2.274533)
       )
-      (stroke (width 0.01) (type solid)) (fill solid) (layer "F.SilkS"))
+      (stroke (width 0.01) (type solid)) (fill solid) (layer "F.Cu"))
     (fp_poly
       (pts
@@
         (xy 1.018309 2.269275)
       )
-      (stroke (width 0.01) (type solid)) (fill solid) (layer "F.SilkS"))
+      (stroke (width 0.01) (type solid)) (fill solid) (layer "F.Cu"))
     (fp_poly
       (pts
@@
         (xy -6.121371 2.269066)
       )
-      (stroke (width 0.01) (type solid)) (fill solid) (layer "F.SilkS"))
+      (stroke (width 0.01) (type solid)) (fill solid) (layer "F.Cu"))
     (fp_poly
       (pts
@@
         (xy -1.300114 2.273448)
       )
-      (stroke (width 0.01) (type solid)) (fill solid) (layer "F.SilkS"))
+      (stroke (width 0.01) (type solid)) (fill solid) (layer "F.Cu"))
     (fp_poly
       (pts
@@
         (xy -1.950081 2.274599)
       )
-      (stroke (width 0.01) (type solid)) (fill solid) (layer "F.SilkS"))
+      (stroke (width 0.01) (type solid)) (fill solid) (layer "F.Cu"))
     (fp_poly
       (pts
@@
         (xy 0.230343 2.26926)
       )
-      (stroke (width 0.01) (type solid)) (fill solid) (layer "F.SilkS"))
+      (stroke (width 0.01) (type solid)) (fill solid) (layer "F.Cu"))
     (fp_poly
       (pts
@@
         (xy -4.712794 2.269146)
       )
-      (stroke (width 0.01) (type solid)) (fill solid) (layer "F.SilkS"))
+      (stroke (width 0.01) (type solid)) (fill solid) (layer "F.Cu"))
     (fp_poly
       (pts
@@
         (xy 3.744665 2.271034)
       )
-      (stroke (width 0.01) (type solid)) (fill solid) (layer "F.SilkS"))
+      (stroke (width 0.01) (type solid)) (fill solid) (layer "F.Cu"))
     (fp_poly
       (pts
@@
         (xy -3.691703 2.270351)
       )
-      (stroke (width 0.01) (type solid)) (fill solid) (layer "F.SilkS"))
+      (stroke (width 0.01) (type solid)) (fill solid) (layer "F.Cu"))
     (fp_poly
       (pts
@@
         (xy 0.328429 -2.050929)
       )
-      (stroke (width 0.01) (type solid)) (fill solid) (layer "F.SilkS"))
+      (stroke (width 0.01) (type solid)) (fill solid) (layer "F.Cu"))
     (fp_poly
       (pts
@@
         (xy 6.186507 -0.527755)
       )
-      (stroke (width 0.01) (type solid)) (fill solid) (layer "F.SilkS"))
+      (stroke (width 0.01) (type solid)) (fill solid) (layer "F.Cu"))
     (fp_poly
       (pts
@@
         (xy 2.673574 -1.133448)
       )
-      (stroke (width 0.01) (type solid)) (fill solid) (layer "F.SilkS"))
+      (stroke (width 0.01) (type solid)) (fill solid) (layer "F.Cu"))
     (fp_poly
       (pts
@@
         (xy -2.9464 -2.510946)
       )
-      (stroke (width 0.01) (type solid)) (fill solid) (layer "F.SilkS"))
+      (stroke (width 0.01) (type solid)) (fill solid) (layer "F.Cu"))
   )
   (footprint "Package_TO_SOT_SMD:SOT-23" (layer "F.Cu")
@@
   )
   (footprint "Symbol:OSHW-Logo_5.7x6mm_Copper" locked (layer "F.Cu")
-    (at 71 51)
+    (at 71 50.6)
     (descr "Open Source Hardware Logo")
     (tags "Logo OSHW")
@@
   (gr_arc (start 94.25 37.5) (mid 93.224874 39.974874) (end 90.75 41)
     (stroke (width 0.1) (type default)) (layer "Margin"))
+  (gr_text "${TITLE} REV ${REVISION}\nhttps://github.com/Alex9779/LoFence\n" (at 71 150.5) (layer "F.Cu")
+    (effects (font (size 1.5 1.5) (thickness 0.25)))
+  )
   (gr_text "On" (at 103.1 61.9506) (layer "F.SilkS")
     (effects (font (size 1.5 1.5) (thickness 0.3)))
@@
     (effects (font (size 1 1) (thickness 0.15)) (justify left bottom))
   )
-  (gr_text "${TITLE} REV ${REVISION}\nhttps://github.com/Alex9779/LoFence\n" (at 71 149.5) (layer "F.SilkS")
-    (effects (font (size 1.3 1.3) (thickness 0.25)))
-  )
   (gr_text "LA" (at 91.7 90.678 90) (layer "F.SilkS")

Commit message: connector updates
- move connectors a little to the inside
- populate ISP connector
Parts:
- moved J5 3.78 mm to (98.4, 85.6)
- moved J6 3.78 mm to (98.4, 90.7)
- moved J3 3.76 mm to (90.8, 75.7)
Routing:
- net MCU_SCK: track 40.6 -> 31.7 mm
- net MCU_MISO: track 49.0 -> 41.0 mm
- net MCU_RESET: track 55.1 -> 47.9 mm
- net +3V3: track 177.0 -> 171.4 mm
- net LA_TX: track 70.0 -> 66.2 mm
- net LA_RX: track 78.0 -> 74.2 mm
- net MCU_MOSI: track 49.6 -> 46.0 mm

Commit message: move DEBUG LED connector and update silkscreen
Parts:
- moved locked 5.54 mm to (87.8, 61.5)
Routing:
- net Net-(D4-K): track 16.0 -> 19.0 mm
Other:
- board text added: "DEBUG LEDs"
Changed lines of the file:
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@@
     (pad_to_mask_clearance 0.2)
     (allow_soldermask_bridges_in_footprints yes)
-    (grid_origin 71 101.5)
+    (grid_origin 85.345 57.912)
     (pcbplotparams
       (layerselection 0x00010f0_ffffffff)
@@
   )
   (footprint "Connector_PinHeader_2.54mm:PinHeader_1x03_P2.54mm_Vertical" (layer "F.Cu")
-    (at 93.3704 61.9252 -90)
+    (at 87.845 61.462 -90)
     (descr "Through hole straight pin header, 1x03, 2.54mm pitch, single row")
     (tags "Through hole pin header THT 1x03 2.54mm single row")
@@
     )
   )
-  (gr_line (start 100.4 63.4506) (end 100.4 60.4506)
+  (gr_line (start 100.4 63.4506) (end 100.4 59.4)
     (stroke (width 0.2) (type solid)) (layer "F.SilkS"))
   (gr_line (start 42 117.5) (end 46 117.5)
     (stroke (width 0.8) (type default)) (layer "F.SilkS"))
+  (gr_line (start 95.1 44.3) (end 80.195 44.3)
+    (stroke (width 0.2) (type default)) (layer "F.SilkS"))
   (gr_rect (start 88.9 77.1913) (end 89.4564 79.2487)
     (stroke (width 0.15) (type solid)) (fill solid) (layer "F.SilkS"))
@@
   (gr_line (start 95.595 79.9245) (end 99.405 79.9245)
     (stroke (width 0.15) (type default)) (layer "F.SilkS"))
+  (gr_line (start 95.1 59.4) (end 80.195 59.4)
+    (stroke (width 0.2) (type default)) (layer "F.SilkS"))
+  (gr_line (start 80.195 44.3) (end 80.195 59.4)
+    (stroke (width 0.2) (type default)) (layer "F.SilkS"))
   (gr_line (start 95.1 59.4) (end 95.1 63.5)
     (stroke (width 0.2) (type default)) (layer "F.SilkS"))
-  (gr_line (start 95.1 60.4) (end 105.7 60.4)
+  (gr_line (start 80.195 59.4) (end 80.195 63.5)
     (stroke (width 0.2) (type default)) (layer "F.SilkS"))
   (gr_line (start 96.2 117.5) (end 100.2 117.5)
     (stroke (width 0.8) (type default)) (layer "F.SilkS"))
+  (gr_line (start 95.1 63.5) (end 80.195 63.5)
+    (stroke (width 0.2) (type default)) (layer "F.SilkS"))
   (gr_line (start 95.1 63.5) (end 105.7 63.5)
     (stroke (width 0.2) (type default)) (layer "F.SilkS"))
@@
     (effects (font (size 1.5 1.5) (thickness 0.25)))
   )
-  (gr_text "On" (at 103.1 61.9506) (layer "F.SilkS")
+  (gr_text "On" (at 103.1 61.562) (layer "F.SilkS")
     (effects (font (size 1.5 1.5) (thickness 0.3)))
   )
@@
     (effects (font (size 1.5 1.5) (thickness 0.3)) (justify left))
   )
-  (gr_text "Off" (at 97.7 61.9506) (layer "F.SilkS")
+  (gr_text "Off" (at 97.7 61.562) (layer "F.SilkS")
     (effects (font (size 1.5 1.5) (thickness 0.3)))
   )
@@
     (effects (font (size 1 1) (thickness 0.15)) (justify left bottom))
   )
+  (gr_text "DEBUG\nLEDs" (at 92.295 62.912) (layer "F.SilkS")
+    (effects (font (size 1 1) (thickness 0.15)) (justify bottom))
+  )
   (gr_text "LA" (at 101.5 90.7 90) (layer "F.SilkS")
     (effects (font (size 1 1) (thickness 0.15)))
@@
   (segment (start 48.0706 79.2877) (end 49.0318 78.3265) (width 0.2) (layer "F.Cu") (net 17))
   (segment (start 93.37 54.912) (end 93.37 57.912) (width 0.2) (layer "F.Cu") (net 18))
-  (segment (start 93.37 57.912) (end 93.37 61.9248) (width 0.2) (layer "F.Cu") (net 18))
+  (segment (start 93.37 57.912) (end 89.82 61.462) (width 0.2) (layer "F.Cu") (net 18))
   (segment (start 93.37 51.912) (end 93.37 54.912) (width 0.2) (layer "F.Cu") (net 18))
   (segment (start 93.37 48.912) (end 93.37 51.912) (width 0.2) (layer "F.Cu") (net 18))
+  (segment (start 89.82 61.462) (end 87.845 61.462) (width 0.2) (layer "F.Cu") (net 18))
   (segment (start 93.37 45.912) (end 93.37 48.912) (width 0.2) (layer "F.Cu") (net 18))
-  (segment (start 93.37 61.9248) (end 93.3704 61.9252) (width 0.2) (layer "F.Cu") (net 18))
   (segment (start 67.8254 65.4084) (end 67.8254 67.15) (width 0.2) (layer "F.Cu") (net 19))
   (via (at 67.8254 65.4084) (size 0.8) (drill 0.4) (layers "F.Cu" "B.Cu") (net 19))
