File: KiCad/LoFence.kicad_pcb (KiCad board)
At the start: 2 copper layers, 72 x 133 mm, 73 parts, among them J1 Fence+, J2 Fence-, J3 ISP, J5 DEBUG MCU, J6 DEBUG LA, J7 FLASH LA, Q1 LBSS84LT1G, Q2 2N7002, U1 TPS63051RMW, U2 TLV9062, U3 ATmega328PB-AU, U4 LA66, Y1 32768 Hz

Commit message: move FLASH LA connector away from case screw hole
Parts:
- moved J7 14.5 mm to (54.5, 69.8), turned to -90 degrees
Routing:
- net LA_BOOT: track 35.5 -> 25.8 mm
- net LA_RESET: track 52.4 -> 45.4 mm
- net LA_RX: track 74.2 -> 79.6 mm
- net LA_TX: track 66.2 -> 68.7 mm
Changed lines of the file:
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@@
     (pad_to_mask_clearance 0.2)
     (allow_soldermask_bridges_in_footprints yes)
-    (grid_origin 100 162.25)
+    (grid_origin 54.8 68.44)
     (pcbplotparams
       (layerselection 0x00010f0_ffffffff)
@@
   )
   (footprint "Connector_PinHeader_2.54mm:PinHeader_1x04_P2.54mm_Vertical" (layer "F.Cu")
-    (at 40.04 69.21)
+    (at 54.536 69.837 -90)
     (descr "Through hole straight pin header, 1x04, 2.54mm pitch, single row")
     (tags "Through hole pin header THT 1x04 2.54mm single row")
@@
     (property "ki_keywords" "connector")
     (attr through_hole exclude_from_bom)
-    (fp_text reference "J7" (at 0 -2.33) (layer "F.SilkS") hide
+    (fp_text reference "J7" (at 0 -2.33 90) (layer "F.SilkS") hide
         (effects (font (size 1 1) (thickness 0.15)))
     )
-    (fp_text value "FLASH LA" (at 0 9.95) (layer "F.Fab")
+    (fp_text value "FLASH LA" (at 0 9.95 90) (layer "F.Fab")
         (effects (font (size 1 1) (thickness 0.15)))
     )
-    (fp_text user "${REFERENCE}" (at 0 3.81 90) (layer "F.Fab")
+    (fp_text user "${REFERENCE}" (at 0 3.81) (layer "F.Fab")
         (effects (font (size 1 1) (thickness 0.15)))
     )
@@
     (fp_line (start 1.27 8.89) (end -1.27 8.89)
       (stroke (width 0.1) (type solid)) (layer "F.Fab"))
-    (pad "1" thru_hole rect (at 0 0) (size 1.7 1.7) (drill 1) (layers "*.Cu" "*.Mask")
+    (pad "1" thru_hole rect (at 0 0 270) (size 1.7 1.7) (drill 1) (layers "*.Cu" "*.Mask")
       (net 56 "LA_BOOT") (pinfunction "Pin_1") (pintype "passive"))
-    (pad "2" thru_hole oval (at 0 2.54) (size 1.7 1.7) (drill 1) (layers "*.Cu" "*.Mask")
+    (pad "2" thru_hole oval (at 0 2.54 270) (size 1.7 1.7) (drill 1) (layers "*.Cu" "*.Mask")
       (net 8 "LA_RX") (pinfunction "Pin_2") (pintype "passive"))
-    (pad "3" thru_hole oval (at 0 5.08) (size 1.7 1.7) (drill 1) (layers "*.Cu" "*.Mask")
+    (pad "3" thru_hole oval (at 0 5.08 270) (size 1.7 1.7) (drill 1) (layers "*.Cu" "*.Mask")
       (net 7 "LA_RESET") (pinfunction "Pin_3") (pintype "passive"))
-    (pad "4" thru_hole oval (at 0 7.62) (size 1.7 1.7) (drill 1) (layers "*.Cu" "*.Mask")
+    (pad "4" thru_hole oval (at 0 7.62 270) (size 1.7 1.7) (drill 1) (layers "*.Cu" "*.Mask")
       (net 1 "GND") (pinfunction "Pin_4") (pintype "passive"))
     (model "${KICAD6_3DMODEL_DIR}/Connector_PinHeader_2.54mm.3dshapes/PinHeader_1x04_P2.54mm_Vertical.wrl" hide
@@
     (effects (font (size 1 1) (thickness 0.15)))
   )
-  (gr_text "FLASH LA" (at 37.85 73.01 90) (layer "F.SilkS")
+  (gr_text "FLASH LA" (at 50.736 67.647) (layer "F.SilkS")
     (effects (font (size 1 1) (thickness 0.15)))
   )
@@
   (segment (start 66.3702 66.294) (end 78.869 66.294) (width 0.2) (layer "B.Cu") (net 6))
   (segment (start 78.869 66.294) (end 90.8 78.225) (width 0.2) (layer "B.Cu") (net 6))
+  (segment (start 49.456 69.837) (end 47.244 67.625) (width 0.2) (layer "F.Cu") (net 7))
   (segment (start 70.2254 64.5095) (end 70.2254 67.15) (width 0.2) (layer "F.Cu") (net 7))
+  (segment (start 47.244 67.625) (end 47.244 62.865) (width 0.2) (layer "F.Cu") (net 7))
   (segment (start 47.244 62.865) (end 68.5809 62.865) (width 0.2) (layer "F.Cu") (net 7))
   (segment (start 38.722 56.515) (end 38.721 56.514) (width 0.2) (layer "F.Cu") (net 7))
@@
   (via (at 40.9194 56.515) (size 0.8) (drill 0.4) (layers "F.Cu" "B.Cu") (net 7))
   (via (at 47.244 62.865) (size 0.8) (drill 0.4) (layers "F.Cu" "B.Cu") (net 7))
-  (segment (start 46.30485 62.865) (end 42.4546 66.71525) (width 0.2) (layer "B.Cu") (net 7))
   (segment (start 47.244 62.8396) (end 40.9194 56.515) (width 0.2) (layer "B.Cu") (net 7))
-  (segment (start 42.4546 66.71525) (end 42.4546 71.8754) (width 0.2) (layer "B.Cu") (net 7))
-  (segment (start 47.244 62.865) (end 46.30485 62.865) (width 0.2) (layer "B.Cu") (net 7))
   (segment (start 47.244 62.865) (end 47.244 62.8396) (width 0.2) (layer "B.Cu") (net 7))
-  (segment (start 42.4546 71.8754) (end 40.04 74.29) (width 0.2) (layer "B.Cu") (net 7))
   (segment (start 43.1546 64.8476) (end 43.146 64.839) (width 0.2) (layer "F.Cu") (net 8))
   (segment (start 72.6186 77.3684) (end 72.6254 77.3616) (width 0.2) (layer "F.Cu") (net 8))
-  (segment (start 43.1546 67.0052) (end 43.1546 68.6354) (width 0.2) (layer "F.Cu") (net 8))
   (segment (start 43.1546 67.0052) (end 43.1546 64.8476) (width 0.2) (layer "F.Cu") (net 8))
-  (segment (start 43.1546 68.6354) (end 40.04 71.75) (width 0.2) (layer "F.Cu") (net 8))
   (segment (start 72.6254 77.3616) (end 72.6254 75.65) (width 0.2) (layer "F.Cu") (net 8))
   (via (at 72.6186 77.3684) (size 0.8) (drill 0.4) (layers "F.Cu" "B.Cu") (net 8))
   (via (at 43.1546 67.0052) (size 0.8) (drill 0.4) (layers "F.Cu" "B.Cu") (net 8))
+  (segment (start 44.061 72.179) (end 43.1546 71.2726) (width 0.2) (layer "B.Cu") (net 8))
+  (segment (start 51.996 69.837) (end 49.643 72.19) (width 0.2) (layer "B.Cu") (net 8))
   (segment (start 72.6186 80.3686) (end 80.8452 88.5952) (width 0.2) (layer "B.Cu") (net 8))
-  (segment (start 72.6186 77.3684) (end 53.5178 77.3684) (width 0.2) (layer "B.Cu") (net 8))
+  (segment (start 49.2504 77.3684) (end 44.061 72.179) (width 0.2) (layer "B.Cu") (net 8))
   (segment (start 93.7772 88.5952) (end 95.86 90.678) (width 0.2) (layer "B.Cu") (net 8))
+  (segment (start 44.072 72.19) (end 44.061 72.179) (width 0.2) (layer "B.Cu") (net 8))
   (segment (start 72.6186 77.3684) (end 72.6186 80.3686) (width 0.2) (layer "B.Cu") (net 8))
-  (segment (start 53.5178 77.3684) (end 43.1546 67.0052) (width 0.2) (layer "B.Cu") (net 8))
+  (segment (start 43.1546 71.2726) (end 43.1546 67.0052) (width 0.2) (layer "B.Cu") (net 8))
+  (segment (start 49.643 72.19) (end 44.072 72.19) (width 0.2) (layer "B.Cu") (net 8))
   (segment (start 80.8452 88.5952) (end 93.7772 88.5952) (width 0.2) (layer "B.Cu") (net 8))
+  (segment (start 72.6186 77.3684) (end 49.2504 77.3684) (width 0.2) (layer "B.Cu") (net 8))
+  (segment (start 44.246 73.3922) (end 44.246 64.839) (width 0.2) (layer "F.Cu") (net 9))
   (segment (start 71.8254 78.0871) (end 71.8312 78.0929) (width 0.2) (layer "F.Cu") (net 9))
-  (segment (start 44.246 69.1888) (end 44.246 64.839) (width 0.2) (layer "F.Cu") (net 9))
-  (segment (start 44.2468 69.1896) (end 44.246 69.1888) (width 0.2) (layer "F.Cu") (net 9))
+  (segment (start 44.2468 73.393) (end 44.246 73.3922) (width 0.2) (layer "F.Cu") (net 9))
   (segment (start 71.8254 75.65) (end 71.8254 78.0871) (width 0.2) (layer "F.Cu") (net 9))
-  (via (at 44.2468 69.1896) (size 0.8) (drill 0.4) (layers "F.Cu" "B.Cu") (net 9))
+  (via (at 44.2468 73.393) (size 0.8) (drill 0.4) (layers "F.Cu" "B.Cu") (net 9))
   (via (at 71.8312 78.0929) (size 0.8) (drill 0.4) (layers "F.Cu" "B.Cu") (net 9))
   (segment (start 71.8312 80.5812) (end 80.6072 89.3572) (width 0.2) (layer "B.Cu") (net 9))
+  (segment (start 44.2468 73.393) (end 48.9467 78.0929) (width 0.2) (layer "B.Cu") (net 9))
   (segment (start 91.9992 89.3572) (end 93.32 90.678) (width 0.2) (layer "B.Cu") (net 9))
-  (segment (start 53.1501 78.0929) (end 44.2468 69.1896) (width 0.2) (layer "B.Cu") (net 9))
-  (segment (start 71.8312 78.0929) (end 53.1501 78.0929) (width 0.2) (layer "B.Cu") (net 9))
+  (segment (start 48.9467 78.0929) (end 71.8312 78.0929) (width 0.2) (layer "B.Cu") (net 9))
   (segment (start 71.8312 78.0929) (end 71.8312 80.5812) (width 0.2) (layer "B.Cu") (net 9))
   (segment (start 80.6072 89.3572) (end 91.9992 89.3572) (width 0.2) (layer "B.Cu") (net 9))
@@
   (segment (start 52.5596 47.4234) (end 52.546 47.4098) (width 0.2) (layer "F.Cu") (net 56))
   (via (at 52.5596 47.4234) (size 0.8) (drill 0.4) (layers "F.Cu" "B.Cu") (net 56))
-  (segment (start 42.4504 47.4234) (end 52.5596 47.4234) (width 0.2) (layer "B.Cu") (net 56))
-  (segment (start 40.01 69.18) (end 40.01 49.8638) (width 0.2) (layer "B.Cu") (net 56))
-  (segment (start 40.01 49.8638) (end 42.4504 47.4234) (width 0.2) (layer "B.Cu") (net 56))
-  (segment (start 40.04 69.21) (end 40.01 69.18) (width 0.2) (layer "B.Cu") (net 56))
+  (segment (start 52.5596 47.4234) (end 54.536 49.3998) (width 0.2) (layer "B.Cu") (net 56))
+  (segment (start 54.536 49.3998) (end 54.536 69.837) (width 0.2) (layer "B.Cu") (net 56))
   (segment (start 82.9313 69.668) (end 82.931 69.6683) (width 0.2) (layer "F.Cu") (net 57))
   (segment (start 92.5556 69.668) (end 85.9556 69.668) (width 0.2) (layer "F.Cu") (net 57))

Commit message: move battery clamps to avoid overlapping with case screw holes
Parts:
- moved B10 0.90 mm to (47.0, 105.6)
- moved B11 0.90 mm to (95.0, 105.6)
- moved B20 0.90 mm to (47.0, 127.6)
- moved B21 0.90 mm to (95.0, 127.6)
- moved B31 0.90 mm to (77.0, 105.6)
- moved B41 0.90 mm to (77.0, 127.6)
- moved D1 0.64 mm to (98.0, 94.6)
Routing:
- net LA_RX: track 79.6 -> 82.6 mm

Commit message: fix DRC
Routing:
- net LA_RX: track 82.6 -> 88.2 mm
Changed lines of the file:
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@@
   (segment (start 44.5 127.6) (end 47 125.1) (width 2.4) (layer "F.Cu") (net 1))
   (segment locked (start 62.38 143.256) (end 57.792 143.256) (width 1.2) (layer "F.Cu") (net 1))
-  (segment (start 39.4 91.2) (end 39.4 105.6) (width 2.4) (layer "F.Cu") (net 1))
   (segment (start 39.4 105.6) (end 39.4 127.6) (width 2.4) (layer "F.Cu") (net 1))
   (segment (start 44.5 105.6) (end 47 108.1) (width 2.4) (layer "F.Cu") (net 1))
@@
   (segment (start 39.4 127.6) (end 44.5 127.6) (width 2.4) (layer "F.Cu") (net 1))
   (segment (start 39.4 105.6) (end 44.5 105.6) (width 2.4) (layer "F.Cu") (net 1))
+  (segment (start 39.4 105.6) (end 39.4 91.2) (width 2.4) (layer "F.Cu") (net 1))
   (segment (start 81.7371 85.8496) (end 81.7371 86.7776) (width 0.27) (layer "F.Cu") (net 1))
   (segment (start 102.9188 65.968) (end 96.3188 65.968) (width 0.2) (layer "F.Cu") (net 1))
@@
   (segment (start 72.6186 77.3684) (end 72.6186 80.3686) (width 0.2) (layer "B.Cu") (net 8))
   (segment (start 43.1546 71.2726) (end 43.1546 67.0052) (width 0.2) (layer "B.Cu") (net 8))
+  (segment (start 44.072 72.19) (end 44.061 72.179) (width 0.2) (layer "B.Cu") (net 8))
   (segment (start 49.2504 77.3684) (end 43.738919 71.856918) (width 0.2) (layer "B.Cu") (net 8))
+  (segment (start 49.643 72.19) (end 44.072 72.19) (width 0.2) (layer "B.Cu") (net 8))
   (segment (start 80.8452 88.5952) (end 93.7772 88.5952) (width 0.2) (layer "B.Cu") (net 8))
   (segment (start 72.6186 77.3684) (end 49.2504 77.3684) (width 0.2) (layer "B.Cu") (net 8))
